File: Simple Audio Amplifier/TDA7053A Stereo.brd (EAGLE design)
At the start: 100 x 80 mm, 16 parts, among them IC1 TDA7052A, IC2 TDA7053A

Commit message: Amplifiers
Parts:
- removed IC2: TDA7053A, My Library:DIL16
- added C4: 1u, SparkFun:CAP-PTH-SMALL2
- added C5, C6: 0.47u, SparkFun:CAP-PTH-SMALL2
- added C8: 0.1u, SparkFun:CAP-PTH-SMALL2
- added R5: 56k, adafruit:0204/5
- added TRIM: 25k, adafruit:TC33X
- added VR: 1M, My Library:POT_ALPHA_RV16AF-20
- added VR1: 22k, My Library:POT_ALPHA_RV16AF-20
- C1: value 100u -> 220u
- C2: value 100n -> 0.1u
- U$1: value 4k7 -> TDA7053A; device My Library:POT_ALPHA_RV16AF-20 -> My Library:DIL16
- moved U$1 54.8 mm to (68.6, 55.9)
- moved JP4 30.6 mm to (22.9, 53.3)
- moved R2 23.6 mm to (24.1, 34.3), turned to 0 degrees
- moved JP3 19.1 mm to (41.9, 53.3)
- moved C3 19.1 mm to (43.2, 47.0), turned to 180 degrees
- moved C1 16.7 mm to (22.9, 44.5)
- moved R1 11.5 mm to (69.8, 36.8)
- moved JP2 11.4 mm to (71.1, 29.2)
- moved R3 11.4 mm to (72.4, 33.0)
- moved C2 8.98 mm to (24.1, 39.4), turned to 180 degrees
- moved IC1 8.89 mm to (33.0, 43.2)
- turned JP1 to 90 degrees
Connections:
- new net AGND: C1.2, C2.2, C4.2, IC1.3, IC1.6, JP3.2, JP4.2, R2.1, VR.1
- new net N$13: C3.2, TRIM.3
- new net N$14: C6.2, U$1.6
- new net N$15: C5.2, U$1.4
- new net N$16: C8.1, R5.1, VR1.3
- new net N$19: U$1.2, U$1.8, VR1.2
- net GND: now also C8.2, U$1.10, U$1.14, U$1.7, VR1.1; no longer C1.2, C2.2, IC1.3, IC1.6, IC2.1, IC2.10, IC2.14, IC2.7, JP3.2, JP4.2, U$1.1
- net N$10: now also U$1.12; no longer IC2.12
- net N$11: now also U$1.13; no longer IC2.13
- net N$12: now also U$1.16; no longer IC2.16
- net N$17: now also R5.2, U$1.5; no longer IC2.5
- net N$2: now also TRIM.2; no longer U$1.2
- net N$3: now also TRIM.1; no longer U$1.3
- net N$4: now also C5.1; no longer IC2.2
- net N$5: now also C4.1, IC1.4, VR.2, VR.3; no longer C3.2, R2.1
- net N$6: now also C6.1; no longer IC2.6
- net N$7: now also U$1.9; no longer IC2.9
Routing:
- net AGND: track 0.00 -> 74.4 mm
- net N$19: track 0.00 -> 73.2 mm
- net GND: track 161.6 -> 130.5 mm
- net N$13: track 0.00 -> 28.8 mm
- net N$5: track 3.81 -> 22.9 mm
- net N$16: track 0.00 -> 17.9 mm
- net N$17: track 21.6 -> 37.2 mm
- net N$8: track 23.0 -> 14.1 mm
- net N$9: track 23.2 -> 14.5 mm
- net N$2: track 15.2 -> 9.12 mm
- net N$1: track 13.5 -> 19.1 mm
- net N$15: track 0.00 -> 3.81 mm
- net N$14: track 0.00 -> 3.81 mm
- net N$6: track 13.8 -> 17.6 mm
- net IN: track 5.08 -> 6.88 mm
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
Commit message: Simple Audio Amp
Parts:
- removed C3: 2u2, SparkFun:CPOL-RADIAL-100UF-25V
- removed C4: 1u, SparkFun:CAP-PTH-SMALL2
- removed IC1: TDA7052A, My Library:DIL08
- removed JP1, JP3, JP4: (no value), pinhead:1X02
- removed JP2: (no value), pinhead:1X04
- removed R2: 1k, adafruit:0204/5
- removed R5: 56k, adafruit:0204/5
- removed SP1: SP, My Library:PS12
- removed TRIM: 25k, adafruit:TC33X
- removed VR: 1M, My Library:POT_ALPHA_RV16AF-20
- added J1: POWER_JACKSLT, SparkFun:POWER_JACK_SLOT
- added U1: (no value), SparkFun:AUDIO-JACK
- C1: value 220u -> 0.1u; device SparkFun:CPOL-RADIAL-100UF-25V -> SparkFun:CAP-PTH-SMALL2
- C2: value 0.1u -> 220u; device SparkFun:CAP-PTH-SMALL2 -> SparkFun:CPOL-RADIAL-100UF-25V
- VR1: value 22k -> 1M
- moved C1 33.3 mm to (54.6, 54.6), turned to 90 degrees
- moved C2 30.3 mm to (49.5, 55.9), turned to 0 degrees
- moved C8 26.1 mm to (81.3, 47.0)
- moved VR1 25.3 mm to (81.3, 26.7)
- moved R1 10.8 mm to (62.2, 44.5)
- moved R3 9.16 mm to (67.3, 40.6), turned to 0 degrees
- moved C5 2.84 mm to (64.8, 47.0), turned to 0 degrees
- moved C6 1.27 mm to (72.4, 44.5)
Connections:
- removed net AGND: C1.2, C2.2, C4.2, IC1.3, IC1.6, JP3.2, JP4.2, R2.1, VR.1
- removed net IN: C3.1, JP3.1
- removed net N$1: C1.1, C2.1, IC1.1, JP4.1
- removed net N$13: C3.2, TRIM.3
- removed net N$16: C8.1, R5.1, VR1.3
- removed net N$2: IC1.2, TRIM.2
- removed net N$3: R2.2, TRIM.1
- removed net N$5: C4.1, IC1.4, VR.2, VR.3
- removed net N$8: IC1.8, SP1.P$1
- removed net N$9: IC1.5, SP1.P$2
- net GND: now also C1.2, C2.2, J1.GND@2, U1.SLEEVE; no longer JP1.2, JP2.3, JP2.4
- net N$17: now also C1.1, C2.1, J1.PWR; no longer JP1.1, R5.2
- net N$19: now also C8.1, VR1.3
- net N$4: now also U1.RING; no longer JP2.1
- net N$6: now also U1.TIP; no longer JP2.2
Routing:
- net AGND: track 74.4 -> 0.00 mm
- net N$13: track 28.8 -> 0.00 mm
- net N$5: track 22.9 -> 0.00 mm
- net N$19: track 73.2 -> 50.9 mm
- net GND: track 130.5 -> 150.9 mm
- net N$1: track 19.1 -> 0.00 mm
- net N$16: track 17.9 -> 0.00 mm
- net N$9: track 14.5 -> 0.00 mm
- net N$8: track 14.1 -> 0.00 mm
- net N$2: track 9.12 -> 0.00 mm
- net N$6: track 17.6 -> 9.80 mm
- net N$3: track 7.42 -> 0.00 mm
- net IN: track 6.88 -> 0.00 mm
- net N$17: track 37.2 -> 31.0 mm
- net N$15: track 3.81 -> 5.08 mm
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