File: Jikken/mic preamp.sch (EAGLE design)
At the start: 18 parts, among them IC1 AD822N

Commit message: jikken
Parts:
- removed JP1: (no value), adafruit:PINHD-1X3
- added C6, C8: 100u, SparkFun:CAP_POLPTH1
- added C7: 100u, capacitor-wima:C2.5/4
- added JP2: (no value), SparkFun:M04POLAR
- added R10: 47, My Library:RESISTORPTH-1/6W
- added R11, R15: 22k, My Library:RESISTORPTH-1/6W
- added R12: 220, My Library:RESISTORPTH-1/6W
- added R13: 47k, My Library:RESISTORPTH-1/6W
- added R14: 100, My Library:RESISTORPTH-1/6W
- added R16: 22k, My Library:RESISTORAXIAL-0.3
- added U$2: 20k, My Library:POT-RV16AF-20
- R6: value 65k -> 68k
- R8: value 50k -> 47k
Connections:
- new net N$10: R12.1, U$2.E, U$2.S
- new net N$11: C6.-, R12.2
- new net N$12: C6.+, IC1B.IN-, R11.1
- new net N$14: IC1B.OUT, R10.1, R11.2
- new net N$15: C8.-, R15.2, U1.RIGHT
- new net N$16: C7.2, R10.2
- new net N$17: C7.1, JP2.3, R13.2
- new net N$18: C8.+, R14.1, R16.1
- new net N$19: IC1B.IN+, R14.2
- net GND: now also JP2.1, R13.1, R15.1, U$2.A; no longer JP1.3
- net N$13: now also JP2.2; no longer JP1.2
- net N$9: now also R16.2
- net VCC: now also JP2.4; no longer JP1.1
Other:
- moved on the sheet: C3
