File: Jikken/Op-amp Microphone Preamp single-supply.sch (EAGLE design)
At the start: 17 parts, among them IC1 AD822N

Commit message: jikken amp
Parts:
- added C2: 0.1uF, SparkFun:CAPKIT
- C1, C4: value 100u -> 100uF/25V
- R1, R5, R7: value 22k -> 22.1k
- R2: value 47k -> 49.9
- R3: value 220 -> 221
- R4: value 68k -> 64.9k
Connections:
- net GND: now also C2.2
- net VCC: now also C2.1
Other:
- moved on the sheet: LOG, R3, R5
Changed lines of the file:
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@@
 <parts>
 <part name="IC1" library="analog-devices" deviceset="AD822" device="N"/>
-<part name="R1" library="My Library" deviceset="RESISTOR" device="PTH-1/6W" value="22k"/>
-<part name="R3" library="My Library" deviceset="RESISTOR" device="PTH-1/6W" value="220"/>
-<part name="C1" library="SparkFun" deviceset="CAP_POL" device="PTH1" value="100u"/>
-<part name="R5" library="My Library" deviceset="RESISTOR" device="PTH-1/6W" value="22k"/>
+<part name="R1" library="My Library" deviceset="RESISTOR" device="PTH-1/6W" value="22.1k"/>
+<part name="R3" library="My Library" deviceset="RESISTOR" device="PTH-1/6W" value="221"/>
+<part name="C1" library="SparkFun" deviceset="CAP_POL" device="PTH1" value="100uF/25V"/>
+<part name="R5" library="My Library" deviceset="RESISTOR" device="PTH-1/6W" value="22.1k"/>
 <part name="U1" library="SparkFun" deviceset="AUDIO-JACK" device="PTH"/>
-<part name="R7" library="My Library" deviceset="RESISTOR" device="PTH-1/6W" value="22k"/>
+<part name="R7" library="My Library" deviceset="RESISTOR" device="PTH-1/6W" value="22.1k"/>
 <part name="P+1" library="SparkFun" deviceset="VCC" device=""/>
 <part name="P+2" library="SparkFun" deviceset="VCC" device=""/>
@@
 <part name="GND6" library="SparkFun" deviceset="GND" device=""/>
 <part name="JP2" library="SparkFun" deviceset="M04" device="POLAR"/>
-<part name="C4" library="SparkFun" deviceset="CAP_POL" device="PTH1" value="100u"/>
+<part name="C4" library="SparkFun" deviceset="CAP_POL" device="PTH1" value="100uF/25V"/>
 <part name="P+3" library="SparkFun" deviceset="VCC" device=""/>
 <part name="LOG" library="My Library" deviceset="POT" device="-RV16AF-20" value="2.5k"/>
-<part name="R2" library="My Library" deviceset="RESISTOR" device="PTH-1/6W" value="47k"/>
-<part name="R4" library="My Library" deviceset="RESISTOR" device="PTH-1/6W" value="68k"/>
+<part name="R2" library="My Library" deviceset="RESISTOR" device="PTH-1/6W" value="49.9"/>
+<part name="R4" library="My Library" deviceset="RESISTOR" device="PTH-1/6W" value="64.9k"/>
 <part name="GND2" library="SparkFun" deviceset="GND" device=""/>
 <part name="C3" library="SparkFun" deviceset="CAP_POL" device="PTH1" value="10u"/>
@@
 <part name="R6" library="My Library" deviceset="RESISTOR" device="PTH-1/6W" value="47"/>
 <part name="R8" library="My Library" deviceset="RESISTOR" device="PTH-1/6W" value="47k"/>
+<part name="C2" library="SparkFun" deviceset="CAP" device="KIT" value="0.1uF"/>
 </parts>
 <sheets>
@@
 <instance part="IC1" gate="A" x="55.88" y="55.88"/>
 <instance part="R1" gate="G$1" x="63.5" y="45.72"/>
-<instance part="R3" gate="G$1" x="40.64" y="40.64" rot="R90"/>
+<instance part="R3" gate="G$1" x="38.1" y="40.64" rot="R90"/>
 <instance part="C1" gate="G$1" x="48.26" y="45.72" rot="R270"/>
-<instance part="R5" gate="G$1" x="27.94" y="43.18" rot="R90"/>
+<instance part="R5" gate="G$1" x="25.4" y="43.18" rot="R90"/>
 <instance part="U1" gate="G$1" x="7.62" y="60.96"/>
 <instance part="R7" gate="G$1" x="40.64" y="71.12" rot="R90"/>
@@
 <instance part="C4" gate="G$1" x="83.82" y="55.88" rot="R90"/>
 <instance part="P+3" gate="1" x="78.74" y="91.44"/>
-<instance part="LOG" gate="G$1" x="40.64" y="27.94"/>
+<instance part="LOG" gate="G$1" x="38.1" y="27.94"/>
 <instance part="R2" gate="G$1" x="27.94" y="76.2" rot="R90"/>
 <instance part="R4" gate="G$1" x="48.26" y="81.28" rot="R180"/>
@@
 <instance part="R6" gate="G$1" x="76.2" y="55.88"/>
 <instance part="R8" gate="G$1" x="88.9" y="38.1" rot="R90"/>
+<instance part="C2" gate="G$1" x="88.9" y="83.82"/>
 </instances>
 <busses>
@@
 <pinref part="GND6" gate="1" pin="GND"/>
 <wire x1="78.74" y1="78.74" x2="78.74" y2="81.28" width="0.1524" layer="91"/>
+<pinref part="C2" gate="G$1" pin="2"/>
+<wire x1="78.74" y1="78.74" x2="88.9" y2="78.74" width="0.1524" layer="91"/>
+<wire x1="88.9" y1="78.74" x2="88.9" y2="81.28" width="0.1524" layer="91"/>
 </segment>
 <segment>
@@
 <wire x1="88.9" y1="33.02" x2="88.9" y2="22.86" width="0.1524" layer="91"/>
 <pinref part="R5" gate="G$1" pin="1"/>
-<wire x1="27.94" y1="22.86" x2="27.94" y2="38.1" width="0.1524" layer="91"/>
+<wire x1="25.4" y1="22.86" x2="25.4" y2="38.1" width="0.1524" layer="91"/>
 <wire x1="15.24" y1="22.86" x2="15.24" y2="63.5" width="0.1524" layer="91"/>
 <pinref part="U1" gate="G$1" pin="SLEEVE"/>
 <wire x1="15.24" y1="63.5" x2="12.7" y2="63.5" width="0.1524" layer="91"/>
 <pinref part="LOG" gate="G$1" pin="A"/>
-<wire x1="40.64" y1="22.86" x2="27.94" y2="22.86" width="0.1524" layer="91"/>
-<wire x1="15.24" y1="22.86" x2="27.94" y2="22.86" width="0.1524" layer="91"/>
-<junction x="27.94" y="22.86"/>
+<wire x1="38.1" y1="22.86" x2="25.4" y2="22.86" width="0.1524" layer="91"/>
+<wire x1="15.24" y1="22.86" x2="25.4" y2="22.86" width="0.1524" layer="91"/>
+<junction x="25.4" y="22.86"/>
 <pinref part="IC1" gate="P" pin="V-"/>
 <wire x1="58.42" y1="48.26" x2="58.42" y2="22.86" width="0.1524" layer="91"/>
-<wire x1="40.64" y1="22.86" x2="58.42" y2="22.86" width="0.1524" layer="91"/>
+<wire x1="38.1" y1="22.86" x2="58.42" y2="22.86" width="0.1524" layer="91"/>
 <wire x1="58.42" y1="22.86" x2="88.9" y2="22.86" width="0.1524" layer="91"/>
 <pinref part="GND5" gate="1" pin="GND"/>
@@
 <wire x1="88.9" y1="22.86" x2="99.06" y2="22.86" width="0.1524" layer="91"/>
 <junction x="58.42" y="22.86"/>
-<junction x="40.64" y="22.86"/>
+<junction x="38.1" y="22.86"/>
 <junction x="88.9" y="22.86"/>
 <junction x="99.06" y="22.86"/>
@@
 <pinref part="P+3" gate="1" pin="VCC"/>
 <wire x1="78.74" y1="91.44" x2="78.74" y2="88.9" width="0.1524" layer="91"/>
+<pinref part="C2" gate="G$1" pin="1"/>
+<wire x1="88.9" y1="88.9" x2="88.9" y2="91.44" width="0.1524" layer="91"/>
+<wire x1="88.9" y1="91.44" x2="78.74" y2="91.44" width="0.1524" layer="91"/>
 </segment>
 </net>
@@
 <pinref part="U1" gate="G$1" pin="LEFT"/>
 <pinref part="R5" gate="G$1" pin="2"/>
-<wire x1="27.94" y1="48.26" x2="27.94" y2="50.8" width="0.1524" layer="91"/>
-<wire x1="27.94" y1="50.8" x2="27.94" y2="58.42" width="0.1524" layer="91"/>
-<wire x1="30.48" y1="58.42" x2="27.94" y2="58.42" width="0.1524" layer="91"/>
-<wire x1="12.7" y1="58.42" x2="27.94" y2="58.42" width="0.1524" layer="91"/>
+<wire x1="25.4" y1="48.26" x2="25.4" y2="50.8" width="0.1524" layer="91"/>
+<wire x1="25.4" y1="50.8" x2="25.4" y2="58.42" width="0.1524" layer="91"/>
+<wire x1="30.48" y1="58.42" x2="25.4" y2="58.42" width="0.1524" layer="91"/>
+<wire x1="12.7" y1="58.42" x2="25.4" y2="58.42" width="0.1524" layer="91"/>
 <pinref part="C6" gate="G$1" pin="-"/>
-<junction x="27.94" y="58.42"/>
+<junction x="25.4" y="58.42"/>
 </segment>
 </net>
@@
 <segment>
 <pinref part="LOG" gate="G$1" pin="S"/>
-<wire x1="45.72" y1="33.02" x2="40.64" y2="33.02" width="0.1524" layer="91"/>
+<wire x1="43.18" y1="33.02" x2="38.1" y2="33.02" width="0.1524" layer="91"/>
 <pinref part="LOG" gate="G$1" pin="E"/>
 <pinref part="R3" gate="G$1" pin="1"/>
-<wire x1="40.64" y1="33.02" x2="45.72" y2="33.02" width="0.1524" layer="91"/>
-<wire x1="45.72" y1="33.02" x2="45.72" y2="27.94" width="0.1524" layer="91"/>
-<junction x="40.64" y="33.02"/>
-<wire x1="40.64" y1="33.02" x2="40.64" y2="35.56" width="0.1524" layer="91"/>
+<wire x1="38.1" y1="33.02" x2="43.18" y2="33.02" width="0.1524" layer="91"/>
+<wire x1="43.18" y1="33.02" x2="43.18" y2="27.94" width="0.1524" layer="91"/>
+<junction x="38.1" y="33.02"/>
+<wire x1="38.1" y1="33.02" x2="38.1" y2="35.56" width="0.1524" layer="91"/>
 </segment>
 </net>
@@
 <pinref part="R3" gate="G$1" pin="2"/>
 <pinref part="C1" gate="G$1" pin="-"/>
-<wire x1="40.64" y1="45.72" x2="43.18" y2="45.72" width="0.1524" layer="91"/>
-</segment>
-</net>
+<wire x1="38.1" y1="45.72" x2="43.18" y2="45.72" width="0.1524" layer="91"/>
+</segment>
+</net>
