File: Jikken/Op-amp Microphone Preamp single-supply.sch (EAGLE design)
At the start: 18 parts, among them IC1 AD822N

Commit message: Amp
Changed lines of the file:
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@@
 <part name="U1" library="SparkFun" deviceset="AUDIO-JACK" device="PTH"/>
 <part name="R7" library="My Library" deviceset="RESISTOR" device="PTH-1/6W" value="22.1k"/>
-<part name="P+1" library="SparkFun" deviceset="VCC" device=""/>
+<part name="P+1" library="SparkFun" deviceset="5V" device=""/>
 <part name="P+2" library="SparkFun" deviceset="VCC" device=""/>
 <part name="GND5" library="SparkFun" deviceset="GND" device=""/>
@@
 <part name="JP2" library="SparkFun" deviceset="M04" device="POLAR"/>
 <part name="C4" library="SparkFun" deviceset="CAP_POL" device="PTH1" value="100uF/25V"/>
-<part name="P+3" library="SparkFun" deviceset="VCC" device=""/>
+<part name="P+3" library="SparkFun" deviceset="5V" device=""/>
 <part name="LOG" library="My Library" deviceset="POT" device="-RV16AF-20" value="2.5k"/>
 <part name="R2" library="My Library" deviceset="RESISTOR" device="PTH-1/6W" value="49.9"/>
@@
 <instance part="R7" gate="G$1" x="40.64" y="71.12" rot="R90"/>
 <instance part="IC1" gate="P" x="58.42" y="55.88" smashed="yes"/>
-<instance part="P+1" gate="1" x="58.42" y="91.44"/>
+<instance part="P+1" gate="G$1" x="58.42" y="91.44"/>
 <instance part="P+2" gate="1" x="99.06" y="68.58"/>
 <instance part="GND5" gate="1" x="99.06" y="22.86"/>
@@
 <instance part="JP2" gate="G$1" x="106.68" y="58.42" rot="MR0"/>
 <instance part="C4" gate="G$1" x="83.82" y="55.88" rot="R90"/>
-<instance part="P+3" gate="1" x="78.74" y="91.44"/>
+<instance part="P+3" gate="G$1" x="78.74" y="91.44"/>
 <instance part="LOG" gate="G$1" x="30.48" y="35.56" rot="MR0"/>
 <instance part="R2" gate="G$1" x="27.94" y="76.2" rot="R90"/>
@@
 <net name="VCC" class="0">
 <segment>
-<pinref part="P+1" gate="1" pin="VCC"/>
+<pinref part="P+1" gate="G$1" pin="5V"/>
 <wire x1="58.42" y1="73.66" x2="58.42" y2="81.28" width="0.1524" layer="91"/>
 <pinref part="IC1" gate="P" pin="V+"/>
@@
 <segment>
 <pinref part="C5" gate="G$1" pin="+"/>
-<pinref part="P+3" gate="1" pin="VCC"/>
+<pinref part="P+3" gate="G$1" pin="5V"/>
 <wire x1="78.74" y1="91.44" x2="78.74" y2="88.9" width="0.1524" layer="91"/>
 <pinref part="C2" gate="G$1" pin="1"/>
