File: Jikken/Amp.brd (EAGLE design)
At the start: 100 x 80 mm, 17 parts, among them IC1 LF356N, U1 INPUT, U2 OUTPUT

Commit message: Amp
Parts:
- moved R1 9.67 mm to (39.4, 39.4)
- moved C4 9.25 mm to (48.3, 47.0), turned to 0 degrees
- moved C2 8.13 mm to (48.3, 43.2), turned to 0 degrees
- moved JP1 7.73 mm to (64.8, 47.0)
- moved R7 6.48 mm to (41.9, 47.0)
- moved R5 6.35 mm to (27.9, 39.4)
- moved R6 6.35 mm to (25.4, 39.4)
- moved R8 4.58 mm to (49.5, 39.4)
- moved U1 4.02 mm to (19.1, 45.7), turned to 0 degrees
- moved R3 2.84 mm to (47.0, 57.1), turned to 90 degrees
- moved C5 2.54 mm to (30.5, 38.1)
- moved C1 2.54 mm to (26.7, 49.5)
- moved C3 2.54 mm to (34.3, 38.1)
- moved U2 2.54 mm to (54.6, 52.1)
- moved R4 1.27 mm to (30.5, 52.1)
Routing:
- net N$1: track 12.0 -> 18.9 mm
- net N$9: track 21.6 -> 15.6 mm
- net VCC: track 38.7 -> 44.3 mm
- net N$7: track 25.5 -> 20.2 mm
- net N$2: track 5.84 -> 10.9 mm
- net N$5: track 23.2 -> 27.4 mm
- net -15V: track 15.5 -> 12.7 mm
- net GND: track 69.6 -> 67.0 mm
- net N$12: track 16.5 -> 15.0 mm
- net N$6: track 1.27 -> 2.54 mm
- net N$4: track 14.0 -> 14.7 mm

Commit message: Amp
Parts:
- C2, C3: value (none) -> 10u
- C4, C5: value (none) -> 0.1u
- R1: value (none) -> 220
- R3, R8: value (none) -> 10
- R4, R5, R6: value (none) -> 2k2
- R7: value (none) -> 200k
- U$1: value (none) -> 20k
- turned C3 to 90 degrees
Connections:
- net GND: now also C3.+; no longer C3.-
- net N$5: now also C3.-; no longer C3.+
Changed lines of the file:
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@@
 <elements>
 <element name="IC1" library="linear" package="DIL08" value="LF356N" x="39.37" y="53.34" rot="R270"/>
-<element name="R1" library="rcl" package="0204/5" value="" x="39.37" y="39.37" rot="R90"/>
-<element name="R3" library="rcl" package="0204/5" value="" x="46.99" y="57.15" rot="R90"/>
-<element name="R4" library="rcl" package="0204/5" value="" x="30.48" y="52.07"/>
-<element name="R5" library="rcl" package="0204/5" value="" x="27.94" y="39.37" rot="R90"/>
-<element name="R6" library="rcl" package="0204/5" value="" x="25.4" y="39.37" rot="R90"/>
-<element name="R8" library="rcl" package="0204/5" value="" x="49.53" y="39.37"/>
+<element name="R1" library="rcl" package="0204/5" value="220" x="39.37" y="39.37" rot="R90"/>
+<element name="R3" library="rcl" package="0204/5" value="10" x="46.99" y="57.15" rot="R90"/>
+<element name="R4" library="rcl" package="0204/5" value="2k2" x="30.48" y="52.07"/>
+<element name="R5" library="rcl" package="0204/5" value="2k2" x="27.94" y="39.37" rot="R90"/>
+<element name="R6" library="rcl" package="0204/5" value="2k2" x="25.4" y="39.37" rot="R90"/>
+<element name="R8" library="rcl" package="0204/5" value="10" x="49.53" y="39.37"/>
 <element name="C1" library="rcl" package="E1,8-4" value="" x="26.67" y="49.53" rot="R180"/>
-<element name="C2" library="rcl" package="E1,8-4" value="" x="48.26" y="43.18"/>
-<element name="C3" library="rcl" package="E1,8-4" value="" x="34.29" y="38.1" rot="R270"/>
-<element name="C4" library="rcl" package="C025-024X044" value="" x="48.26" y="46.99"/>
-<element name="C5" library="rcl" package="C025-024X044" value="" x="30.48" y="38.1" rot="R270"/>
-<element name="U$1" library="SparkFun" package="3362U" value="" x="35.56" y="60.96"/>
-<element name="R7" library="rcl" package="0204/5" value="" x="41.91" y="46.99"/>
+<element name="C2" library="rcl" package="E1,8-4" value="10u" x="48.26" y="43.18"/>
+<element name="C3" library="rcl" package="E1,8-4" value="10u" x="34.29" y="38.1" rot="R90"/>
+<element name="C4" library="rcl" package="C025-024X044" value="0.1u" x="48.26" y="46.99"/>
+<element name="C5" library="rcl" package="C025-024X044" value="0.1u" x="30.48" y="38.1" rot="R270"/>
+<element name="U$1" library="SparkFun" package="3362U" value="20k" x="35.56" y="60.96"/>
+<element name="R7" library="rcl" package="0204/5" value="200k" x="41.91" y="46.99"/>
 <element name="U1" library="SparkFun" package="STEREOJACK2.5MM_SPECIAL_HOLES-ONLY" value="INPUT" x="19.05" y="45.72"/>
 <element name="JP1" library="SparkFun" package="MOLEX-1X4" value="POWER" x="64.77" y="46.99" rot="R270"/>
@@
 <signal name="GND">
 <contactref element="C5" pad="2"/>
-<contactref element="C3" pad="-"/>
 <contactref element="R5" pad="1"/>
 <contactref element="R6" pad="1"/>
@@
 <wire x1="22.86" y1="36.83" x2="25.4" y2="36.83" width="0.4064" layer="16"/>
 <wire x1="30.48" y1="36.83" x2="34.29" y2="36.83" width="0.254" layer="1"/>
-<wire x1="34.29" y1="36.83" x2="34.29" y2="37.211" width="0.254" layer="1"/>
 <wire x1="34.29" y1="36.83" x2="39.37" y2="36.83" width="0.254" layer="1"/>
-<wire x1="34.29" y1="36.83" x2="34.29" y2="37.211" width="0.254" layer="1"/>
 <wire x1="30.48" y1="36.83" x2="27.94" y2="36.83" width="0.254" layer="1"/>
 <wire x1="49.53" y1="46.99" x2="49.53" y2="43.18" width="0.254" layer="1"/>
@@
 <wire x1="39.37" y1="36.83" x2="49.53" y2="36.83" width="0.4064" layer="16"/>
 <wire x1="49.53" y1="36.83" x2="49.53" y2="43.18" width="0.4064" layer="16"/>
-<wire x1="49.53" y1="43.18" x2="49.149" y2="43.18" width="0" layer="19" extent="1-16"/>
 <wire x1="49.53" y1="46.99" x2="49.53" y2="49.53" width="0.4064" layer="16"/>
 <wire x1="49.53" y1="49.53" x2="52.76" y2="49.53" width="0.4064" layer="16"/>
 <wire x1="52.76" y1="49.53" x2="52.76" y2="49.57" width="0.4064" layer="16"/>
+<contactref element="C3" pad="+"/>
+<wire x1="34.29" y1="36.83" x2="34.29" y2="37.211" width="0.254" layer="1"/>
 </signal>
 <signal name="N$1">
@@
 <signal name="N$5">
 <contactref element="IC1" pad="4"/>
-<contactref element="C3" pad="+"/>
 <contactref element="C5" pad="1"/>
 <contactref element="R8" pad="1"/>
 <wire x1="30.48" y1="39.37" x2="34.29" y2="39.37" width="0.254" layer="1"/>
-<wire x1="34.29" y1="39.37" x2="34.29" y2="38.989" width="0.254" layer="1"/>
 <wire x1="34.29" y1="39.37" x2="35.56" y2="39.37" width="0.254" layer="1"/>
 <wire x1="35.56" y1="39.37" x2="46.99" y2="39.37" width="0.254" layer="1"/>
+<wire x1="35.56" y1="39.37" x2="35.56" y2="49.53" width="0.254" layer="1"/>
+<contactref element="C3" pad="-"/>
 <wire x1="34.29" y1="39.37" x2="34.29" y2="38.989" width="0.254" layer="1"/>
-<wire x1="35.56" y1="39.37" x2="35.56" y2="49.53" width="0.254" layer="1"/>
 </signal>
 <signal name="N$13">

Commit message: jikken
Parts:
- moved C2 16.6 mm to (49.5, 59.7)
- moved C4 7.73 mm to (49.5, 54.6)
- moved C3 6.84 mm to (40.6, 40.6)
- moved R1 6.84 mm to (45.7, 41.9)
- moved C5 5.68 mm to (35.6, 40.6)
- moved U2 3.81 mm to (58.4, 52.1), turned to 180 degrees
- moved R4 3.59 mm to (33.0, 49.5), turned to 90 degrees
- moved R5 3.59 mm to (30.5, 41.9)
- moved R8 2.84 mm to (50.8, 41.9)
- moved C1 2.54 mm to (29.2, 49.5)
- moved JP1 2.54 mm to (64.8, 49.5)
- moved R6 2.54 mm to (25.4, 41.9)
- moved R3 1.27 mm to (45.7, 57.1)
- moved R7 1.27 mm to (43.2, 47.0)
Routing:
- net GND: track 66.7 -> 96.8 mm
- net VCC: track 44.3 -> 50.1 mm
- net N$9: track 15.6 -> 10.2 mm
- net N$7: track 20.2 -> 24.1 mm
- net N$5: track 27.1 -> 29.2 mm
- net N$2: track 10.9 -> 9.43 mm
- net -15V: track 12.7 -> 11.4 mm
- net N$4: track 14.7 -> 15.9 mm

Commit message: Amp
Parts:
- C1: value (none) -> 10u
- R7: value 200k -> 220k
- U$1: device SparkFun:3362U -> My Library:3362U
Changed lines of the file:
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@@
 <layer number="106" name="bPlate" color="7" fill="1" visible="no" active="yes"/>
 <layer number="107" name="Crop" color="7" fill="1" visible="no" active="yes"/>
+<layer number="108" name="fp8" color="7" fill="1" visible="no" active="yes"/>
+<layer number="109" name="fp9" color="7" fill="1" visible="no" active="yes"/>
+<layer number="110" name="fp0" color="7" fill="1" visible="no" active="yes"/>
 <layer number="116" name="Patch_BOT" color="9" fill="4" visible="no" active="yes"/>
 <layer number="121" name="_tsilk" color="7" fill="1" visible="no" active="yes"/>
 <layer number="122" name="_bsilk" color="7" fill="1" visible="no" active="yes"/>
+<layer number="123" name="tTestmark" color="7" fill="1" visible="no" active="yes"/>
+<layer number="124" name="bTestmark" color="7" fill="1" visible="no" active="yes"/>
 <layer number="125" name="_tNames" color="7" fill="1" visible="no" active="yes"/>
+<layer number="131" name="tAdjust" color="7" fill="1" visible="no" active="yes"/>
+<layer number="132" name="bAdjust" color="7" fill="1" visible="no" active="yes"/>
 <layer number="144" name="Drill_legend" color="7" fill="1" visible="no" active="yes"/>
 <layer number="151" name="HeatSink" color="7" fill="1" visible="no" active="yes"/>
+<layer number="199" name="Contour" color="7" fill="1" visible="yes" active="yes"/>
 <layer number="200" name="200bmp" color="1" fill="10" visible="no" active="yes"/>
 <layer number="201" name="201bmp" color="2" fill="10" visible="no" active="yes"/>
@@
 <element name="R6" library="rcl" package="0204/5" value="2k2" x="25.4" y="41.91" rot="R90"/>
 <element name="R8" library="rcl" package="0204/5" value="10" x="50.8" y="41.91"/>
-<element name="C1" library="rcl" package="E1,8-4" value="" x="29.21" y="49.53" rot="R180"/>
+<element name="C1" library="rcl" package="E1,8-4" value="10u" x="29.21" y="49.53" rot="R180"/>
 <element name="C2" library="rcl" package="E1,8-4" value="10u" x="49.53" y="59.69"/>
 <element name="C3" library="rcl" package="E1,8-4" value="10u" x="40.64" y="40.64" rot="R90"/>
 <element name="C4" library="rcl" package="C025-024X044" value="0.1u" x="49.53" y="54.61"/>
 <element name="C5" library="rcl" package="C025-024X044" value="0.1u" x="35.56" y="40.64" rot="R270"/>
-<element name="U$1" library="SparkFun" package="3362U" value="20k" x="35.56" y="60.96"/>
-<element name="R7" library="rcl" package="0204/5" value="200k" x="43.18" y="46.99"/>
+<element name="U$1" library="My Library" package="3362U" value="20k" x="35.56" y="60.96"/>
+<element name="R7" library="rcl" package="0204/5" value="220k" x="43.18" y="46.99"/>
 <element name="U1" library="SparkFun" package="STEREOJACK2.5MM_SPECIAL_HOLES-ONLY" value="INPUT" x="19.05" y="45.72"/>
 <element name="JP1" library="SparkFun" package="MOLEX-1X4" value="POWER" x="64.77" y="49.53" rot="R270"/>
