File: Jikken/Amp.sch (EAGLE design)
At the start: 17 parts, among them IC1 LF356N, U1 INPUT, U2 OUTPUT

Commit message: Amp
Parts:
- C2, C3: value (none) -> 10u
- C4, C5: value (none) -> 0.1u
- R1: value (none) -> 220
- R3, R8: value (none) -> 10
- R4, R5, R6: value (none) -> 2k2
- R7: value (none) -> 200k
- U$1: value (none) -> 20k
Connections:
- net GND: now also C3.+; no longer C3.-
- net N$5: now also C3.-; no longer C3.+
Other:
- moved on the sheet: C1, C3, C5, R6, U1
Changed lines of the file:
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@@
 <parts>
 <part name="IC1" library="linear" deviceset="LF356" device="N"/>
-<part name="R1" library="rcl" deviceset="R-EU_" device="0204/5"/>
-<part name="R3" library="rcl" deviceset="R-EU_" device="0204/5"/>
-<part name="R4" library="rcl" deviceset="R-EU_" device="0204/5"/>
-<part name="R5" library="rcl" deviceset="R-EU_" device="0204/5"/>
-<part name="R6" library="rcl" deviceset="R-EU_" device="0204/5"/>
-<part name="R8" library="rcl" deviceset="R-EU_" device="0204/5"/>
+<part name="R1" library="rcl" deviceset="R-EU_" device="0204/5" value="220"/>
+<part name="R3" library="rcl" deviceset="R-EU_" device="0204/5" value="10"/>
+<part name="R4" library="rcl" deviceset="R-EU_" device="0204/5" value="2k2"/>
+<part name="R5" library="rcl" deviceset="R-EU_" device="0204/5" value="2k2"/>
+<part name="R6" library="rcl" deviceset="R-EU_" device="0204/5" value="2k2"/>
+<part name="R8" library="rcl" deviceset="R-EU_" device="0204/5" value="10"/>
 <part name="C1" library="rcl" deviceset="CPOL-EU" device="E1.8-4"/>
-<part name="C2" library="rcl" deviceset="CPOL-EU" device="E1.8-4"/>
-<part name="C3" library="rcl" deviceset="CPOL-EU" device="E1.8-4"/>
-<part name="C4" library="rcl" deviceset="C-EU" device="025-024X044"/>
-<part name="C5" library="rcl" deviceset="C-EU" device="025-024X044"/>
+<part name="C2" library="rcl" deviceset="CPOL-EU" device="E1.8-4" value="10u"/>
+<part name="C3" library="rcl" deviceset="CPOL-EU" device="E1.8-4" value="10u"/>
+<part name="C4" library="rcl" deviceset="C-EU" device="025-024X044" value="0.1u"/>
+<part name="C5" library="rcl" deviceset="C-EU" device="025-024X044" value="0.1u"/>
 <part name="SUPPLY4" library="supply2" deviceset="GND" device=""/>
 <part name="SUPPLY5" library="supply2" deviceset="GND" device=""/>
@@
 <part name="SUPPLY9" library="supply2" deviceset="GND" device=""/>
 <part name="SUPPLY10" library="supply2" deviceset="GND" device=""/>
-<part name="U$1" library="SparkFun" deviceset="POT" device="100K_3362U"/>
-<part name="R7" library="rcl" deviceset="R-EU_" device="0204/5"/>
+<part name="U$1" library="SparkFun" deviceset="POT" device="100K_3362U" value="20k"/>
+<part name="R7" library="rcl" deviceset="R-EU_" device="0204/5" value="200k"/>
 <part name="U1" library="SparkFun" deviceset="AUDIO-JACK" device="HOLESONLY" value="INPUT"/>
 <part name="JP1" library="SparkFun" deviceset="M04" device="POLAR" value="POWER"/>
@@
 <instance part="R4" gate="G$1" x="45.72" y="76.2"/>
 <instance part="R5" gate="G$1" x="36.83" y="68.58" rot="R90"/>
-<instance part="R6" gate="G$1" x="22.86" y="68.58" rot="R90"/>
+<instance part="R6" gate="G$1" x="27.94" y="68.58" rot="R90"/>
 <instance part="R8" gate="G$1" x="58.42" y="46.99" rot="R270"/>
-<instance part="C1" gate="G$1" x="30.48" y="76.2" rot="R270"/>
+<instance part="C1" gate="G$1" x="33.02" y="76.2" rot="R270"/>
 <instance part="C2" gate="G$1" x="48.26" y="91.44"/>
-<instance part="C3" gate="G$1" x="50.8" y="49.53"/>
+<instance part="C3" gate="G$1" x="48.26" y="46.99" rot="MR180"/>
 <instance part="C4" gate="G$1" x="40.64" y="91.44"/>
-<instance part="C5" gate="G$1" x="43.18" y="49.53"/>
-<instance part="SUPPLY4" gate="GND" x="50.8" y="39.37"/>
-<instance part="SUPPLY5" gate="GND" x="43.18" y="39.37"/>
+<instance part="C5" gate="G$1" x="40.64" y="49.53"/>
+<instance part="SUPPLY4" gate="GND" x="48.26" y="39.37"/>
+<instance part="SUPPLY5" gate="GND" x="40.64" y="39.37"/>
 <instance part="P+2" gate="VCC" x="58.42" y="111.76"/>
 <instance part="P-1" gate="1" x="58.42" y="33.02"/>
 <instance part="SUPPLY1" gate="GND" x="36.83" y="59.69"/>
-<instance part="SUPPLY2" gate="GND" x="22.86" y="59.69"/>
-<instance part="SUPPLY3" gate="GND" x="15.24" y="69.85"/>
+<instance part="SUPPLY2" gate="GND" x="27.94" y="59.69"/>
+<instance part="SUPPLY3" gate="GND" x="20.32" y="64.77"/>
 <instance part="SUPPLY6" gate="GND" x="73.66" y="44.45"/>
 <instance part="SUPPLY9" gate="GND" x="40.64" y="83.82"/>
@@
 <instance part="U$1" gate="G$1" x="68.58" y="86.36" rot="R90"/>
 <instance part="R7" gate="G$1" x="73.66" y="66.04" rot="R90"/>
-<instance part="U1" gate="G$1" x="2.54" y="78.74"/>
+<instance part="U1" gate="G$1" x="10.16" y="78.74"/>
 <instance part="JP1" gate="G$1" x="104.14" y="96.52" rot="R180"/>
 <instance part="P+1" gate="VCC" x="88.9" y="109.22"/>
@@
 <net name="GND" class="0">
 <segment>
-<wire x1="43.18" y1="44.45" x2="43.18" y2="41.91" width="0.1524" layer="91"/>
+<wire x1="40.64" y1="44.45" x2="40.64" y2="41.91" width="0.1524" layer="91"/>
 <pinref part="SUPPLY5" gate="GND" pin="GND"/>
 <pinref part="C5" gate="G$1" pin="2"/>
-</segment>
-<segment>
-<wire x1="50.8" y1="44.45" x2="50.8" y2="41.91" width="0.1524" layer="91"/>
-<pinref part="SUPPLY4" gate="GND" pin="GND"/>
-<pinref part="C3" gate="G$1" pin="-"/>
 </segment>
 <segment>
@@
 </segment>
 <segment>
-<wire x1="22.86" y1="63.5" x2="22.86" y2="62.23" width="0.1524" layer="91"/>
+<wire x1="27.94" y1="63.5" x2="27.94" y2="62.23" width="0.1524" layer="91"/>
 <pinref part="R6" gate="G$1" pin="1"/>
 <pinref part="SUPPLY2" gate="GND" pin="GND"/>
 </segment>
 <segment>
-<wire x1="15.24" y1="72.39" x2="15.24" y2="81.28" width="0.1524" layer="91"/>
+<wire x1="20.32" y1="67.31" x2="20.32" y2="81.28" width="0.1524" layer="91"/>
 <pinref part="SUPPLY3" gate="GND" pin="GND"/>
 <pinref part="U1" gate="G$1" pin="SLEEVE"/>
-<wire x1="15.24" y1="81.28" x2="7.62" y2="81.28" width="0.1524" layer="91"/>
+<wire x1="20.32" y1="81.28" x2="15.24" y2="81.28" width="0.1524" layer="91"/>
 </segment>
 <segment>
@@
 <pinref part="SUPPLY7" gate="GND" pin="GND"/>
 </segment>
+<segment>
+<pinref part="SUPPLY4" gate="GND" pin="GND"/>
+<wire x1="48.26" y1="41.91" x2="48.26" y2="44.45" width="0.1524" layer="91"/>
+<pinref part="C3" gate="G$1" pin="+"/>
+</segment>
 </net>
 <net name="N$1" class="0">
 <segment>
-<wire x1="22.86" y1="73.66" x2="22.86" y2="76.2" width="0.1524" layer="91"/>
-<wire x1="7.62" y1="76.2" x2="22.86" y2="76.2" width="0.1524" layer="91"/>
-<wire x1="22.86" y1="76.2" x2="25.4" y2="76.2" width="0.1524" layer="91"/>
-<junction x="22.86" y="76.2"/>
+<wire x1="27.94" y1="73.66" x2="27.94" y2="76.2" width="0.1524" layer="91"/>
+<wire x1="15.24" y1="76.2" x2="27.94" y2="76.2" width="0.1524" layer="91"/>
+<junction x="27.94" y="76.2"/>
 <pinref part="R6" gate="G$1" pin="2"/>
 <pinref part="C1" gate="G$1" pin="-"/>
@@
 <net name="N$2" class="0">
 <segment>
-<wire x1="33.02" y1="76.2" x2="36.83" y2="76.2" width="0.1524" layer="91"/>
+<wire x1="35.56" y1="76.2" x2="36.83" y2="76.2" width="0.1524" layer="91"/>
 <wire x1="36.83" y1="76.2" x2="40.64" y2="76.2" width="0.1524" layer="91"/>
 <wire x1="36.83" y1="73.66" x2="36.83" y2="76.2" width="0.1524" layer="91"/>
@@
 <wire x1="58.42" y1="66.04" x2="58.42" y2="55.88" width="0.1524" layer="91"/>
 <wire x1="58.42" y1="52.07" x2="58.42" y2="55.88" width="0.1524" layer="91"/>
-<wire x1="58.42" y1="55.88" x2="50.8" y2="55.88" width="0.1524" layer="91"/>
-<wire x1="43.18" y1="52.07" x2="43.18" y2="55.88" width="0.1524" layer="91"/>
-<wire x1="43.18" y1="55.88" x2="50.8" y2="55.88" width="0.1524" layer="91"/>
-<wire x1="50.8" y1="55.88" x2="50.8" y2="52.07" width="0.1524" layer="91"/>
-<junction x="50.8" y="55.88"/>
+<wire x1="58.42" y1="55.88" x2="48.26" y2="55.88" width="0.1524" layer="91"/>
+<wire x1="40.64" y1="52.07" x2="40.64" y2="55.88" width="0.1524" layer="91"/>
+<wire x1="40.64" y1="55.88" x2="48.26" y2="55.88" width="0.1524" layer="91"/>
 <junction x="58.42" y="55.88"/>
 <pinref part="IC1" gate="A" pin="V-"/>
-<pinref part="C3" gate="G$1" pin="+"/>
 <pinref part="C5" gate="G$1" pin="1"/>
 <pinref part="R8" gate="G$1" pin="1"/>
-</segment>
-</net>
+<pinref part="C3" gate="G$1" pin="-"/>
+<wire x1="48.26" y1="52.07" x2="48.26" y2="55.88" width="0.1524" layer="91"/>
+</segment>
+</net>

Commit message: Amp
Parts:
- C1: value (none) -> 10u
- R7: value 200k -> 220k
- U$1: device SparkFun:POT100K_3362U -> My Library:POT100K_3362U
Other:
- moved on the sheet: U$1
Changed lines of the file:
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@@
 <layer number="106" name="bPlate" color="7" fill="1" visible="no" active="yes"/>
 <layer number="107" name="Crop" color="7" fill="1" visible="no" active="yes"/>
+<layer number="108" name="fp8" color="7" fill="1" visible="no" active="yes"/>
+<layer number="109" name="fp9" color="7" fill="1" visible="no" active="yes"/>
+<layer number="110" name="fp0" color="7" fill="1" visible="no" active="yes"/>
 <layer number="116" name="Patch_BOT" color="9" fill="4" visible="no" active="yes"/>
 <layer number="121" name="_tsilk" color="7" fill="1" visible="no" active="yes"/>
 <layer number="122" name="_bsilk" color="7" fill="1" visible="no" active="yes"/>
+<layer number="123" name="tTestmark" color="7" fill="1" visible="no" active="yes"/>
+<layer number="124" name="bTestmark" color="7" fill="1" visible="no" active="yes"/>
 <layer number="125" name="_tNames" color="7" fill="1" visible="no" active="yes"/>
+<layer number="131" name="tAdjust" color="7" fill="1" visible="no" active="yes"/>
+<layer number="132" name="bAdjust" color="7" fill="1" visible="no" active="yes"/>
 <layer number="144" name="Drill_legend" color="7" fill="1" visible="no" active="yes"/>
 <layer number="151" name="HeatSink" color="7" fill="1" visible="no" active="yes"/>
+<layer number="199" name="Contour" color="7" fill="1" visible="yes" active="yes"/>
 <layer number="200" name="200bmp" color="1" fill="10" visible="no" active="yes"/>
 <layer number="201" name="201bmp" color="2" fill="10" visible="no" active="yes"/>
@@
 <part name="R6" library="rcl" deviceset="R-EU_" device="0204/5" value="2k2"/>
 <part name="R8" library="rcl" deviceset="R-EU_" device="0204/5" value="10"/>
-<part name="C1" library="rcl" deviceset="CPOL-EU" device="E1.8-4"/>
+<part name="C1" library="rcl" deviceset="CPOL-EU" device="E1.8-4" value="10u"/>
 <part name="C2" library="rcl" deviceset="CPOL-EU" device="E1.8-4" value="10u"/>
 <part name="C3" library="rcl" deviceset="CPOL-EU" device="E1.8-4" value="10u"/>
@@
 <part name="SUPPLY9" library="supply2" deviceset="GND" device=""/>
 <part name="SUPPLY10" library="supply2" deviceset="GND" device=""/>
-<part name="U$1" library="SparkFun" deviceset="POT" device="100K_3362U" value="20k"/>
-<part name="R7" library="rcl" deviceset="R-EU_" device="0204/5" value="200k"/>
+<part name="U$1" library="My Library" deviceset="POT" device="100K_3362U" value="20k"/>
+<part name="R7" library="rcl" deviceset="R-EU_" device="0204/5" value="220k"/>
 <part name="U1" library="SparkFun" deviceset="AUDIO-JACK" device="HOLESONLY" value="INPUT"/>
 <part name="JP1" library="SparkFun" deviceset="M04" device="POLAR" value="POWER"/>
@@
 <instance part="SUPPLY9" gate="GND" x="40.64" y="83.82"/>
 <instance part="SUPPLY10" gate="GND" x="48.26" y="83.82"/>
-<instance part="U$1" gate="G$1" x="68.58" y="86.36" rot="R90"/>
+<instance part="U$1" gate="G$1" x="68.58" y="81.28" rot="R90"/>
 <instance part="R7" gate="G$1" x="73.66" y="66.04" rot="R90"/>
 <instance part="U1" gate="G$1" x="10.16" y="78.74"/>
@@
 <net name="VCC" class="0">
 <segment>
-<wire x1="68.58" y1="91.44" x2="68.58" y2="101.6" width="0.1524" layer="91"/>
+<wire x1="68.58" y1="86.36" x2="68.58" y2="101.6" width="0.1524" layer="91"/>
 <wire x1="68.58" y1="101.6" x2="68.58" y2="106.68" width="0.1524" layer="91"/>
 <wire x1="68.58" y1="106.68" x2="58.42" y2="106.68" width="0.1524" layer="91"/>
@@
 <net name="N$13" class="0">
 <segment>
-<wire x1="60.96" y1="86.36" x2="60.96" y2="81.28" width="0.1524" layer="91"/>
+<wire x1="63.5" y1="81.28" x2="60.96" y2="81.28" width="0.1524" layer="91"/>
 <pinref part="IC1" gate="A" pin="ON1"/>
 <pinref part="U$1" gate="G$1" pin="E"/>
@@
 <segment>
 <wire x1="68.58" y1="76.2" x2="73.66" y2="76.2" width="0.1524" layer="91"/>
-<wire x1="73.66" y1="76.2" x2="76.2" y2="76.2" width="0.1524" layer="91"/>
-<wire x1="76.2" y1="76.2" x2="76.2" y2="86.36" width="0.1524" layer="91"/>
+<wire x1="73.66" y1="76.2" x2="73.66" y2="81.28" width="0.1524" layer="91"/>
 <pinref part="IC1" gate="A" pin="ON2"/>
 <pinref part="U$1" gate="G$1" pin="A"/>
