File: Jikken/Op-amp Microphone Preamp.sch (EAGLE design)
At the start: 29 parts, among them IC1 AD822N

Commit message: Amplifiers
Parts:
- removed C3: 10u, SparkFun:CAP_POLPTH1
- removed C6, C8: 100u, SparkFun:CAP_POLPTH1
- removed C7: 100u, capacitor-wima:C2.5/4
- removed R10, R2: 47, My Library:RESISTORPTH-1/6W
- removed R11, R15: 22k, My Library:RESISTORPTH-1/6W
- removed R12: 220, My Library:RESISTORPTH-1/6W
- removed R13, R8, R9: 47k, My Library:RESISTORPTH-1/6W
- removed R14, R4: 100, My Library:RESISTORPTH-1/6W
- removed R16: 22k, My Library:RESISTORAXIAL-0.3
- removed R6: 68k, My Library:RESISTORPTH-1/6W
- removed U$1, U$2: 20k, My Library:POT-RV16AF-20
- C1, C2: value 100u -> 10u
- C4: value 100u -> 10u; device capacitor-wima:C2.5/4 -> SparkFun:CAP_POLPTH1
- R3: value 220 -> 1k; device My Library:RESISTORPTH-1/6W -> SparkFun:RESISTORPTH-1/4W
- R5: value 22k -> 47k; device My Library:RESISTORPTH-1/6W -> SparkFun:RESISTORPTH-1/4W
- R7: value 22k -> 47k; device My Library:RESISTORAXIAL-0.3 -> SparkFun:RESISTORPTH-1/4W
Connections:
- removed net N$1: R3.1, U$1.E, U$1.S
- removed net N$10: R12.1, U$2.E, U$2.S
- removed net N$11: C6.-, R12.2
- removed net N$12: C6.+, IC1B.IN-, R11.1
- removed net N$14: IC1B.OUT, R10.1, R11.2
- removed net N$15: C8.-, R15.2, U1.RIGHT
- removed net N$16: C7.2, R10.2
- removed net N$17: C7.1, JP2.3, R13.2
- removed net N$18: C8.+, R14.1, R16.1
- removed net N$19: IC1B.IN+, R14.2
- removed net N$4: C4.2, R2.2
- removed net N$7: C2.+, R4.1, R7.1
- net GND: now also JP2.2, R3.1; no longer C3.-, JP2.1, R13.1, R15.1, R8.1, R9.1, U$1.A, U$2.A
- net N$13: now also C4.-, JP2.1; no longer C4.1, JP2.2, R9.2
- net N$3: now also C4.+; no longer R2.1
- net N$6: now also C2.+, IC1A.IN+, R7.1; no longer C2.-, U1.LEFT
- net N$8: now also C2.-, U1.LEFT; no longer IC1A.IN+, R4.2
- net N$9: now also U1.RIGHT; no longer C3.+, R16.2, R6.1, R7.2, R8.2
- net VCC: now also JP2.3, R7.2; no longer JP2.4, R6.2
Other:
- note added: "http://www.zen22142.zen.co.uk/Circuits/Audio/lf071_mic.htm"
- moved on the sheet: C1, C2, C5, JP2, R1, R3, R5, R7, U1

Commit message: Preamp
Parts:
- added C3: 0.1uF, SparkFun:CAPPTH
- added TRIMPOT: 10k, My Library:POT100K_3362U
- IC1: value AD822N -> LF356N; device analog-devices:AD822N -> My Library:LF356N
- R3: value 1k -> 100; device SparkFun:RESISTORPTH-1/4W -> SparkFun:RESISTORPTH-1/6W
- R5, R7: device SparkFun:RESISTORPTH-1/4W -> SparkFun:RESISTORPTH-1/6W
Connections:
- new net N$4: R3.1, TRIMPOT.A, TRIMPOT.S
- net GND: now also C3.2, IC1.V-, TRIMPOT.E; no longer IC1P.V-, R3.1
- net N$3: now also IC1.OUT; no longer IC1A.OUT
- net N$5: now also IC1.-IN; no longer IC1A.IN-
- net N$6: now also IC1.+IN; no longer IC1A.IN+
- net VCC: now also C3.1, IC1.V+; no longer IC1P.V+
Other:
- moved on the sheet: C1, C4, R1, R3, R7
Changed lines of the file:
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@@
 </classes>
 <parts>
-<part name="IC1" library="analog-devices" deviceset="AD822" device="N"/>
 <part name="R1" library="My Library" deviceset="RESISTOR" device="PTH-1/6W" value="22k"/>
-<part name="R3" library="SparkFun" deviceset="RESISTOR" device="PTH-1/4W" value="1k"/>
+<part name="R3" library="SparkFun" deviceset="RESISTOR" device="PTH-1/6W" value="100"/>
 <part name="C1" library="SparkFun" deviceset="CAP_POL" device="PTH1" value="10u"/>
 <part name="GND1" library="SparkFun" deviceset="GND" device=""/>
-<part name="R5" library="SparkFun" deviceset="RESISTOR" device="PTH-1/4W" value="47k"/>
+<part name="R5" library="SparkFun" deviceset="RESISTOR" device="PTH-1/6W" value="47k"/>
 <part name="U1" library="SparkFun" deviceset="AUDIO-JACK" device="PTH"/>
-<part name="R7" library="SparkFun" deviceset="RESISTOR" device="PTH-1/4W" value="47k"/>
+<part name="R7" library="SparkFun" deviceset="RESISTOR" device="PTH-1/6W" value="47k"/>
 <part name="P+1" library="SparkFun" deviceset="VCC" device=""/>
 <part name="GND4" library="SparkFun" deviceset="GND" device=""/>
@@
 <part name="C2" library="SparkFun" deviceset="CAP_POL" device="PTH1" value="10u"/>
 <part name="P+3" library="SparkFun" deviceset="VCC" device=""/>
+<part name="IC1" library="My Library" deviceset="LF356" device="N"/>
+<part name="TRIMPOT" library="My Library" deviceset="POT" device="100K_3362U" value="10k"/>
+<part name="C3" library="SparkFun" deviceset="CAP" device="PTH" value="0.1uF"/>
 </parts>
 <sheets>
@@
 </plain>
 <instances>
-<instance part="IC1" gate="A" x="55.88" y="50.8"/>
-<instance part="R1" gate="G$1" x="66.04" y="40.64"/>
-<instance part="R3" gate="G$1" x="40.64" y="33.02" rot="R90"/>
-<instance part="C1" gate="G$1" x="48.26" y="40.64" rot="R270"/>
-<instance part="GND1" gate="1" x="40.64" y="20.32"/>
+<instance part="R1" gate="G$1" x="71.12" y="40.64"/>
+<instance part="R3" gate="G$1" x="43.18" y="40.64"/>
+<instance part="C1" gate="G$1" x="55.88" y="40.64" rot="R270"/>
+<instance part="GND1" gate="1" x="15.24" y="20.32"/>
 <instance part="R5" gate="G$1" x="30.48" y="48.26" rot="R90"/>
 <instance part="U1" gate="G$1" x="7.62" y="55.88"/>
-<instance part="R7" gate="G$1" x="40.64" y="63.5" rot="R90"/>
-<instance part="IC1" gate="P" x="58.42" y="50.8" smashed="yes"/>
-<instance part="P+1" gate="1" x="58.42" y="78.74"/>
-<instance part="GND4" gate="1" x="58.42" y="20.32"/>
+<instance part="R7" gate="G$1" x="50.8" y="63.5" rot="R90"/>
+<instance part="P+1" gate="1" x="63.5" y="78.74"/>
+<instance part="GND4" gate="1" x="63.5" y="20.32"/>
 <instance part="P+2" gate="1" x="91.44" y="60.96"/>
 <instance part="GND5" gate="1" x="91.44" y="20.32"/>
 <instance part="C5" gate="G$1" x="111.76" y="78.74"/>
-<instance part="GND6" gate="1" x="111.76" y="68.58"/>
+<instance part="GND6" gate="1" x="111.76" y="66.04"/>
 <instance part="JP2" gate="G$1" x="104.14" y="53.34" rot="MR0"/>
-<instance part="C4" gate="G$1" x="78.74" y="50.8" rot="R90"/>
+<instance part="C4" gate="G$1" x="81.28" y="50.8" rot="R90"/>
 <instance part="C2" gate="G$1" x="22.86" y="53.34" rot="R270"/>
 <instance part="P+3" gate="1" x="111.76" y="86.36"/>
+<instance part="IC1" gate="G$1" x="66.04" y="50.8"/>
+<instance part="TRIMPOT" gate="G$1" x="38.1" y="27.94" rot="R90"/>
+<instance part="C3" gate="G$1" x="121.92" y="76.2"/>
 </instances>
 <busses>
@@
 <segment>
 <pinref part="R1" gate="G$1" pin="2"/>
-<wire x1="71.12" y1="40.64" x2="71.12" y2="50.8" width="0.1524" layer="91"/>
-<pinref part="IC1" gate="A" pin="OUT"/>
-<wire x1="71.12" y1="50.8" x2="66.04" y2="50.8" width="0.1524" layer="91"/>
-<wire x1="71.12" y1="50.8" x2="76.2" y2="50.8" width="0.1524" layer="91"/>
-<junction x="71.12" y="50.8"/>
+<wire x1="76.2" y1="40.64" x2="76.2" y2="50.8" width="0.1524" layer="91"/>
+<wire x1="76.2" y1="50.8" x2="73.66" y2="50.8" width="0.1524" layer="91"/>
+<wire x1="76.2" y1="50.8" x2="78.74" y2="50.8" width="0.1524" layer="91"/>
+<junction x="76.2" y="50.8"/>
 <pinref part="C4" gate="G$1" pin="+"/>
+<pinref part="IC1" gate="G$1" pin="OUT"/>
 </segment>
 </net>
 <net name="N$5" class="0">
 <segment>
-<pinref part="IC1" gate="A" pin="IN-"/>
 <pinref part="C1" gate="G$1" pin="+"/>
-<wire x1="50.8" y1="48.26" x2="50.8" y2="40.64" width="0.1524" layer="91"/>
+<wire x1="58.42" y1="48.26" x2="58.42" y2="40.64" width="0.1524" layer="91"/>
 <pinref part="R1" gate="G$1" pin="1"/>
-<wire x1="50.8" y1="40.64" x2="60.96" y2="40.64" width="0.1524" layer="91"/>
-<junction x="50.8" y="40.64"/>
+<wire x1="58.42" y1="40.64" x2="66.04" y2="40.64" width="0.1524" layer="91"/>
+<junction x="58.42" y="40.64"/>
+<pinref part="IC1" gate="G$1" pin="-IN"/>
 </segment>
 </net>
@@
 <pinref part="R3" gate="G$1" pin="2"/>
 <pinref part="C1" gate="G$1" pin="-"/>
-<wire x1="40.64" y1="38.1" x2="40.64" y2="40.64" width="0.1524" layer="91"/>
-<wire x1="40.64" y1="40.64" x2="43.18" y2="40.64" width="0.1524" layer="91"/>
+<wire x1="48.26" y1="40.64" x2="50.8" y2="40.64" width="0.1524" layer="91"/>
 </segment>
 </net>
 <net name="GND" class="0">
 <segment>
-<pinref part="IC1" gate="P" pin="V-"/>
 <pinref part="GND4" gate="1" pin="GND"/>
-<wire x1="58.42" y1="43.18" x2="58.42" y2="22.86" width="0.1524" layer="91"/>
+<wire x1="63.5" y1="43.18" x2="63.5" y2="22.86" width="0.1524" layer="91"/>
+<pinref part="IC1" gate="G$1" pin="V-"/>
 </segment>
 <segment>
@@
 <pinref part="C5" gate="G$1" pin="-"/>
 <pinref part="GND6" gate="1" pin="GND"/>
+<wire x1="111.76" y1="68.58" x2="111.76" y2="71.12" width="0.1524" layer="91"/>
+<pinref part="C3" gate="G$1" pin="2"/>
 <wire x1="111.76" y1="71.12" x2="111.76" y2="73.66" width="0.1524" layer="91"/>
+<wire x1="111.76" y1="71.12" x2="121.92" y2="71.12" width="0.1524" layer="91"/>
+<wire x1="121.92" y1="71.12" x2="121.92" y2="73.66" width="0.1524" layer="91"/>
+<junction x="111.76" y="71.12"/>
 </segment>
 <segment>
-<pinref part="GND1" gate="1" pin="GND"/>
 <pinref part="R5" gate="G$1" pin="1"/>
 <wire x1="30.48" y1="27.94" x2="30.48" y2="43.18" width="0.1524" layer="91"/>
@@
 <wire x1="15.24" y1="45.72" x2="15.24" y2="58.42" width="0.1524" layer="91"/>
 <wire x1="15.24" y1="58.42" x2="12.7" y2="58.42" width="0.1524" layer="91"/>
-<wire x1="30.48" y1="27.94" x2="40.64" y2="27.94" width="0.1524" layer="91"/>
+<pinref part="TRIMPOT" gate="G$1" pin="E"/>
+<wire x1="30.48" y1="27.94" x2="33.02" y2="27.94" width="0.1524" layer="91"/>
+<wire x1="15.24" y1="27.94" x2="15.24" y2="22.86" width="0.1524" layer="91"/>
+<pinref part="GND1" gate="1" pin="GND"/>
+<junction x="15.24" y="27.94"/>
 <junction x="30.48" y="27.94"/>
-<wire x1="40.64" y1="22.86" x2="40.64" y2="27.94" width="0.1524" layer="91"/>
-<pinref part="R3" gate="G$1" pin="1"/>
-<junction x="40.64" y="27.94"/>
 </segment>
 </net>
@@
 <segment>
 <pinref part="R5" gate="G$1" pin="2"/>
-<wire x1="30.48" y1="53.34" x2="40.64" y2="53.34" width="0.1524" layer="91"/>
+<wire x1="30.48" y1="53.34" x2="50.8" y2="53.34" width="0.1524" layer="91"/>
 <pinref part="R7" gate="G$1" pin="1"/>
-<wire x1="40.64" y1="58.42" x2="40.64" y2="53.34" width="0.1524" layer="91"/>
-<wire x1="40.64" y1="53.34" x2="50.8" y2="53.34" width="0.1524" layer="91"/>
-<pinref part="IC1" gate="A" pin="IN+"/>
+<wire x1="50.8" y1="58.42" x2="50.8" y2="53.34" width="0.1524" layer="91"/>
+<wire x1="50.8" y1="53.34" x2="58.42" y2="53.34" width="0.1524" layer="91"/>
 <pinref part="C2" gate="G$1" pin="+"/>
 <junction x="30.48" y="53.34"/>
-<junction x="40.64" y="53.34"/>
+<junction x="50.8" y="53.34"/>
 <wire x1="30.48" y1="53.34" x2="25.4" y2="53.34" width="0.1524" layer="91"/>
+<pinref part="IC1" gate="G$1" pin="+IN"/>
 </segment>
 </net>
@@
 <segment>
 <pinref part="P+1" gate="1" pin="VCC"/>
-<wire x1="58.42" y1="73.66" x2="58.42" y2="78.74" width="0.1524" layer="91"/>
-<pinref part="IC1" gate="P" pin="V+"/>
-<wire x1="58.42" y1="58.42" x2="58.42" y2="73.66" width="0.1524" layer="91"/>
+<wire x1="63.5" y1="68.58" x2="63.5" y2="78.74" width="0.1524" layer="91"/>
+<wire x1="63.5" y1="58.42" x2="63.5" y2="68.58" width="0.1524" layer="91"/>
 <pinref part="R7" gate="G$1" pin="2"/>
-<wire x1="40.64" y1="68.58" x2="40.64" y2="73.66" width="0.1524" layer="91"/>
-<wire x1="40.64" y1="73.66" x2="58.42" y2="73.66" width="0.1524" layer="91"/>
-<junction x="58.42" y="73.66"/>
+<wire x1="50.8" y1="68.58" x2="63.5" y2="68.58" width="0.1524" layer="91"/>
+<junction x="63.5" y="68.58"/>
+<pinref part="IC1" gate="G$1" pin="V+"/>
 </segment>
 <segment>
@@
 <pinref part="C5" gate="G$1" pin="+"/>
 <pinref part="P+3" gate="1" pin="VCC"/>
-<wire x1="111.76" y1="86.36" x2="111.76" y2="81.28" width="0.1524" layer="91"/>
+<wire x1="111.76" y1="86.36" x2="111.76" y2="83.82" width="0.1524" layer="91"/>
+<pinref part="C3" gate="G$1" pin="1"/>
+<wire x1="111.76" y1="83.82" x2="111.76" y2="81.28" width="0.1524" layer="91"/>
+<wire x1="121.92" y1="81.28" x2="121.92" y2="83.82" width="0.1524" layer="91"/>
+<wire x1="121.92" y1="83.82" x2="111.76" y2="83.82" width="0.1524" layer="91"/>
+<junction x="111.76" y="83.82"/>
 </segment>
 </net>
 <net name="N$13" class="0">
 <segment>
-<wire x1="91.44" y1="50.8" x2="83.82" y2="50.8" width="0.1524" layer="91"/>
+<wire x1="91.44" y1="50.8" x2="86.36" y2="50.8" width="0.1524" layer="91"/>
 <wire x1="91.44" y1="50.8" x2="96.52" y2="50.8" width="0.1524" layer="91"/>
 <wire x1="96.52" y1="50.8" x2="99.06" y2="50.8" width="0.1524" layer="91"/>
@@
 </segment>
 </net>
+<net name="N$4" class="0">
+<segment>
+<pinref part="R3" gate="G$1" pin="1"/>
+<pinref part="TRIMPOT" gate="G$1" pin="S"/>
+<wire x1="38.1" y1="40.64" x2="38.1" y2="33.02" width="0.1524" layer="91"/>
+<wire x1="38.1" y1="33.02" x2="45.72" y2="33.02" width="0.1524" layer="91"/>
+<wire x1="45.72" y1="33.02" x2="45.72" y2="27.94" width="0.1524" layer="91"/>
+<pinref part="TRIMPOT" gate="G$1" pin="A"/>
+<wire x1="45.72" y1="27.94" x2="43.18" y2="27.94" width="0.1524" layer="91"/>
+<junction x="38.1" y="33.02"/>
+</segment>
+</net>

Commit message: Amp
Parts:
- R5: value 47k -> 22k
- R7: value 47k -> 68k
Changed lines of the file:
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@@
 <part name="C1" library="SparkFun" deviceset="CAP_POL" device="PTH1" value="10u"/>
 <part name="GND1" library="SparkFun" deviceset="GND" device=""/>
-<part name="R5" library="SparkFun" deviceset="RESISTOR" device="PTH-1/6W" value="47k"/>
+<part name="R5" library="SparkFun" deviceset="RESISTOR" device="PTH-1/6W" value="22k"/>
 <part name="U1" library="SparkFun" deviceset="AUDIO-JACK" device="PTH"/>
-<part name="R7" library="SparkFun" deviceset="RESISTOR" device="PTH-1/6W" value="47k"/>
+<part name="R7" library="SparkFun" deviceset="RESISTOR" device="PTH-1/6W" value="68k"/>
 <part name="P+1" library="SparkFun" deviceset="VCC" device=""/>
 <part name="GND4" library="SparkFun" deviceset="GND" device=""/>
