File: Jikken/plug-board.sch (EAGLE design)
At the start: 19 parts

Commit message: lib
Parts:
- removed D1: 1N4007, JPN:1N4007
- removed DC_POEWR, DC_POEWR1, DC_POEWR2: DCPOWER, My Library:DCPOWER
- removed LOAD, LOAD1: (no value), rcl:R-EU_0204/5
- removed LOAD5: 330, rcl:R-EU_0204/5
- removed U$1, U$3, U$5: AMMETER, My Library:AMMETER
- removed U$2, U$4, U$7: VOLTMETER, My Library:VOLTMETER
- added BAT2: AAA, adafruit:AAA
- added R0: (no value), rcl:R-EU_0204/5
- added SW1: (no value), switch:REKN
- LOAD2: value 50 -> Inf
- LOAD4: value Infinity -> 50
- renumbered BAT to BATTERY
Connections:
- removed net AGND: DC_POEWR.VGND, DC_POEWR1.VGND, DC_POEWR2.VGND
- removed net N$11: D1.A, U$5.P$2, U$7.P$1
- removed net N$12: D1.C, LOAD5.1, U$7.P$2
- removed net N$2: LOAD.1, U$1.P$2, U$2.P$1
- net GND: no longer LOAD.2, LOAD1.2, LOAD5.2, U$2.P$2, U$4.P$2
- net N$1: now also SW1.0@A; no longer DC_POEWR.VOUT, U$1.P$1
- net N$10: now also SW1.1@A; no longer DC_POEWR2.VOUT, U$5.P$1
- net N$3: now also BAT2.-, R0.1; no longer DC_POEWR1.VOUT, U$3.P$1, U$4.P$1
- net N$5: now also R0.2; no longer LOAD1.1, U$3.P$2
Other:
- note added: "J1"
- note added: "J2"
- note added: "J3"
- note added: "J4"
- note added: "L1"
- note added: "L2"
- note added: "L3"
- note added: "L4"
- note added: "L5"
- note added: "L6"
- note added: "L7"
- note added: "L8"
- note added: "P1"
- note added: "P2"
- note added: "T1"
- note added: "T2"
- note added: "T3"
- note removed: "Ammeter"
- note removed: "DC POWER"
- note removed: "LOAD"
