File: Microchip SPI SRAM/23Kxxx.sch (EAGLE design)
At the start: 5 parts, among them IC2 23KP, Q1 BSS101

Commit message: SRAM
Parts:
- added R3, R4, R5, R6, R7, R8, R9: (no value), My Library:RESISTORAXIAL-0.3
- Q1: value BSS101 -> 2SK1772; device transistor-fet:BSS101 -> My Library:2SK1772
Connections:
- removed net N$1: IC2.GND
- new net GND: IC2.GND, JP1.5, R4.1, R6.1, R8.1
- new net N$11: JP1.1, R7.1, R8.2
- new net N$8: JP1.2, R5.1, R6.2
- new net N$9: IC2.SI, R5.2
- net 3.3V: now also IC2.VCC, JP1.7, R9.2
- net 5V: now also JP1.8
- net N$2: now also JP1.3; no longer JP1.4
- net N$4: now also R7.2
- net N$5: now also JP1.6, R9.1
- net N$6: now also R3.2
- net N$7: now also JP1.4, R3.1, R4.2; no longer IC2.SI
Other:
- moved on the sheet: IC2, JP1, R1, R2

Commit message: SPI SRAM pcb layout
Parts:
- R1, R2: value (none) -> 4.7k
- R3, R5, R7: value (none) -> 5.1k
- R4: value (none) -> 7.5
- R6, R8: value (none) -> 7.5k
- R9: value (none) -> 10k
Connections:
- removed net N$2: JP1.3, Q1.S, R1.1
- new net N$1: JP1.3, Q1.D, R1.1
- net N$3: now also Q1.S; no longer Q1.D
Other:
- moved on the sheet: R1, R2
Changed lines of the file:
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@@
 <part name="Q1" library="My Library" deviceset="2SK1772" device=""/>
 <part name="U$2" library="SparkFun" deviceset="5V" device=""/>
-<part name="R2" library="My Library" deviceset="RESISTOR" device="AXIAL-0.3"/>
-<part name="R1" library="My Library" deviceset="RESISTOR" device="AXIAL-0.3"/>
-<part name="R3" library="My Library" deviceset="RESISTOR" device="AXIAL-0.3"/>
-<part name="R4" library="My Library" deviceset="RESISTOR" device="AXIAL-0.3"/>
-<part name="R5" library="My Library" deviceset="RESISTOR" device="AXIAL-0.3"/>
-<part name="R6" library="My Library" deviceset="RESISTOR" device="AXIAL-0.3"/>
-<part name="R7" library="My Library" deviceset="RESISTOR" device="AXIAL-0.3"/>
-<part name="R8" library="My Library" deviceset="RESISTOR" device="AXIAL-0.3"/>
+<part name="R2" library="My Library" deviceset="RESISTOR" device="AXIAL-0.3" value="4.7k"/>
+<part name="R1" library="My Library" deviceset="RESISTOR" device="AXIAL-0.3" value="4.7k"/>
+<part name="R3" library="My Library" deviceset="RESISTOR" device="AXIAL-0.3" value="5.1k"/>
+<part name="R4" library="My Library" deviceset="RESISTOR" device="AXIAL-0.3" value="7.5"/>
+<part name="R5" library="My Library" deviceset="RESISTOR" device="AXIAL-0.3" value="5.1k"/>
+<part name="R6" library="My Library" deviceset="RESISTOR" device="AXIAL-0.3" value="7.5k"/>
+<part name="R7" library="My Library" deviceset="RESISTOR" device="AXIAL-0.3" value="5.1k"/>
+<part name="R8" library="My Library" deviceset="RESISTOR" device="AXIAL-0.3" value="7.5k"/>
 <part name="GND1" library="SparkFun" deviceset="GND" device=""/>
 <part name="GND2" library="SparkFun" deviceset="GND" device=""/>
 <part name="GND3" library="SparkFun" deviceset="GND" device=""/>
 <part name="GND4" library="SparkFun" deviceset="GND" device=""/>
-<part name="R9" library="My Library" deviceset="RESISTOR" device="AXIAL-0.3"/>
+<part name="R9" library="My Library" deviceset="RESISTOR" device="AXIAL-0.3" value="10k"/>
 <part name="GND5" library="SparkFun" deviceset="GND" device=""/>
 <part name="JP1" library="SparkFun" deviceset="M08" device="1X08"/>
@@
 <instances>
 <instance part="IC2" gate="G$1" x="53.34" y="66.04"/>
-<instance part="P+1" gate="G$1" x="30.48" y="96.52"/>
-<instance part="Q1" gate="G$1" x="20.32" y="66.04" rot="R270"/>
+<instance part="P+1" gate="G$1" x="20.32" y="96.52"/>
+<instance part="Q1" gate="G$1" x="20.32" y="66.04" rot="MR270"/>
 <instance part="U$2" gate="G$1" x="12.7" y="96.52"/>
-<instance part="R2" gate="G$1" x="30.48" y="83.82" rot="R90"/>
-<instance part="R1" gate="G$1" x="12.7" y="83.82" rot="R90"/>
+<instance part="R2" gate="G$1" x="30.48" y="81.28" rot="R90"/>
+<instance part="R1" gate="G$1" x="12.7" y="81.28" rot="R90"/>
 <instance part="R3" gate="G$1" x="81.28" y="58.42" rot="R90"/>
 <instance part="R4" gate="G$1" x="81.28" y="45.72" rot="R90"/>
@@
 <instance part="GND4" gate="1" x="53.34" y="35.56"/>
 <instance part="R9" gate="G$1" x="73.66" y="81.28" rot="R90"/>
-<instance part="GND5" gate="1" x="7.62" y="83.82"/>
+<instance part="GND5" gate="1" x="2.54" y="35.56"/>
 <instance part="JP1" gate="G$1" x="-12.7" y="68.58"/>
 <instance part="U$1" gate="G$1" x="-5.08" y="93.98"/>
@@
 <segment>
 <pinref part="IC2" gate="G$1" pin="SO"/>
-<wire x1="27.94" y1="66.04" x2="30.48" y2="66.04" width="0.1524" layer="91"/>
-<pinref part="Q1" gate="G$1" pin="D"/>
 <wire x1="30.48" y1="66.04" x2="40.64" y2="66.04" width="0.1524" layer="91"/>
 <pinref part="R2" gate="G$1" pin="1"/>
-<wire x1="30.48" y1="78.74" x2="30.48" y2="66.04" width="0.1524" layer="91"/>
-<junction x="30.48" y="66.04"/>
+<wire x1="30.48" y1="76.2" x2="30.48" y2="66.04" width="0.1524" layer="91"/>
+<pinref part="Q1" gate="G$1" pin="S"/>
+<wire x1="27.94" y1="66.04" x2="30.48" y2="66.04" width="0.1524" layer="91"/>
 </segment>
 </net>
@@
 <pinref part="R3" gate="G$1" pin="1"/>
 <wire x1="81.28" y1="50.8" x2="81.28" y2="53.34" width="0.1524" layer="91"/>
-<wire x1="81.28" y1="50.8" x2="78.74" y2="50.8" width="0.1524" layer="91"/>
-<wire x1="78.74" y1="50.8" x2="10.16" y2="50.8" width="0.1524" layer="91"/>
+<wire x1="81.28" y1="50.8" x2="10.16" y2="50.8" width="0.1524" layer="91"/>
 <wire x1="10.16" y1="50.8" x2="10.16" y2="68.58" width="0.1524" layer="91"/>
 <wire x1="10.16" y1="68.58" x2="-7.62" y2="68.58" width="0.1524" layer="91"/>
 <pinref part="JP1" gate="G$1" pin="4"/>
-<junction x="78.74" y="50.8"/>
+<junction x="81.28" y="50.8"/>
 </segment>
 </net>
@@
 <segment>
 <pinref part="Q1" gate="G$1" pin="G"/>
-<wire x1="20.32" y1="74.295" x2="20.32" y2="88.9" width="0.1524" layer="91"/>
+<wire x1="20.32" y1="76.2" x2="20.32" y2="91.44" width="0.1524" layer="91"/>
 <pinref part="P+1" gate="G$1" pin="3.3V"/>
-<wire x1="20.32" y1="88.9" x2="30.48" y2="88.9" width="0.1524" layer="91"/>
-<wire x1="30.48" y1="88.9" x2="30.48" y2="91.44" width="0.1524" layer="91"/>
-<pinref part="R2" gate="G$1" pin="2"/>
 <pinref part="IC2" gate="G$1" pin="VCC"/>
-<wire x1="30.48" y1="91.44" x2="30.48" y2="96.52" width="0.1524" layer="91"/>
+<wire x1="20.32" y1="91.44" x2="20.32" y2="96.52" width="0.1524" layer="91"/>
+<wire x1="20.32" y1="91.44" x2="30.48" y2="91.44" width="0.1524" layer="91"/>
 <wire x1="30.48" y1="91.44" x2="53.34" y2="91.44" width="0.1524" layer="91"/>
 <wire x1="53.34" y1="91.44" x2="53.34" y2="78.74" width="0.1524" layer="91"/>
@@
 <wire x1="73.66" y1="86.36" x2="73.66" y2="91.44" width="0.1524" layer="91"/>
 <wire x1="73.66" y1="91.44" x2="53.34" y2="91.44" width="0.1524" layer="91"/>
-<junction x="30.48" y="88.9"/>
+<pinref part="R2" gate="G$1" pin="2"/>
+<wire x1="30.48" y1="86.36" x2="30.48" y2="91.44" width="0.1524" layer="91"/>
+<junction x="30.48" y="91.44"/>
+<junction x="20.32" y="91.44"/>
+<junction x="53.34" y="91.44"/>
 </segment>
 <segment>
@@
 </segment>
 </net>
-<net name="N$2" class="0">
-<segment>
-<wire x1="-7.62" y1="66.04" x2="12.7" y2="66.04" width="0.1524" layer="91"/>
-<wire x1="12.7" y1="66.04" x2="15.24" y2="66.04" width="0.1524" layer="91"/>
-<pinref part="Q1" gate="G$1" pin="S"/>
-<pinref part="R1" gate="G$1" pin="1"/>
-<wire x1="12.7" y1="78.74" x2="12.7" y2="66.04" width="0.1524" layer="91"/>
-<junction x="12.7" y="66.04"/>
-<pinref part="JP1" gate="G$1" pin="3"/>
-</segment>
-</net>
 <net name="5V" class="0">
 <segment>
 <pinref part="U$2" gate="G$1" pin="5V"/>
 <pinref part="R1" gate="G$1" pin="2"/>
-<wire x1="12.7" y1="96.52" x2="12.7" y2="88.9" width="0.1524" layer="91"/>
+<wire x1="12.7" y1="96.52" x2="12.7" y2="86.36" width="0.1524" layer="91"/>
 </segment>
 <segment>
@@
 <segment>
 <wire x1="-7.62" y1="71.12" x2="2.54" y2="71.12" width="0.1524" layer="91"/>
-<wire x1="2.54" y1="71.12" x2="2.54" y2="91.44" width="0.1524" layer="91"/>
+<wire x1="2.54" y1="71.12" x2="2.54" y2="55.88" width="0.1524" layer="91"/>
 <pinref part="GND5" gate="1" pin="GND"/>
-<wire x1="2.54" y1="91.44" x2="7.62" y2="91.44" width="0.1524" layer="91"/>
-<wire x1="7.62" y1="91.44" x2="7.62" y2="86.36" width="0.1524" layer="91"/>
+<wire x1="2.54" y1="55.88" x2="2.54" y2="50.8" width="0.1524" layer="91"/>
+<wire x1="2.54" y1="50.8" x2="2.54" y2="38.1" width="0.1524" layer="91"/>
 <pinref part="JP1" gate="G$1" pin="5"/>
 </segment>
 </net>
+<net name="N$1" class="0">
+<segment>
+<pinref part="JP1" gate="G$1" pin="3"/>
+<pinref part="Q1" gate="G$1" pin="D"/>
+<wire x1="-7.62" y1="66.04" x2="12.7" y2="66.04" width="0.1524" layer="91"/>
+<pinref part="R1" gate="G$1" pin="1"/>
+<wire x1="12.7" y1="66.04" x2="12.7" y2="76.2" width="0.1524" layer="91"/>
+</segment>
+</net>

Commit message: Amp
Changed lines of the file:
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@@
 <instance part="GND5" gate="1" x="2.54" y="35.56"/>
 <instance part="JP1" gate="G$1" x="-12.7" y="68.58"/>
-<instance part="U$1" gate="G$1" x="-5.08" y="93.98"/>
-<instance part="P+2" gate="G$1" x="-2.54" y="88.9"/>
+<instance part="U$1" gate="G$1" x="-5.08" y="96.52"/>
+<instance part="P+2" gate="G$1" x="0" y="96.52"/>
 </instances>
 <busses>
@@
 <segment>
 <pinref part="P+2" gate="G$1" pin="3.3V"/>
-<wire x1="-2.54" y1="88.9" x2="-2.54" y2="76.2" width="0.1524" layer="91"/>
+<wire x1="0" y1="96.52" x2="0" y2="76.2" width="0.1524" layer="91"/>
 <pinref part="JP1" gate="G$1" pin="7"/>
-<wire x1="-2.54" y1="76.2" x2="-7.62" y2="76.2" width="0.1524" layer="91"/>
+<wire x1="0" y1="76.2" x2="-7.62" y2="76.2" width="0.1524" layer="91"/>
 </segment>
 </net>
@@
 <pinref part="U$1" gate="G$1" pin="5V"/>
 <wire x1="-7.62" y1="78.74" x2="-5.08" y2="78.74" width="0.1524" layer="91"/>
-<wire x1="-5.08" y1="78.74" x2="-5.08" y2="93.98" width="0.1524" layer="91"/>
+<wire x1="-5.08" y1="78.74" x2="-5.08" y2="96.52" width="0.1524" layer="91"/>
 </segment>
 </net>
