File: OP amp module/Absolute value circuit.sch (EAGLE design)
At the start: 9 parts, among them IC1 LM358N

Commit message: Op mic-preamp single
Connections:
- net GND renamed +5V/2
Other:
- moved on the sheet: R3
Changed lines of the file:
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@@
 <part name="JP1" library="SparkFun" deviceset="M01" device="PTH"/>
 <part name="JP2" library="SparkFun" deviceset="M01" device="PTH"/>
-<part name="GND1" library="SparkFun" deviceset="GND" device=""/>
+<part name="SUPPLY1" library="supply2" deviceset="+5V/2" device=""/>
 </parts>
 <sheets>
@@
 <instance part="R1" gate="G$1" x="66.04" y="45.72"/>
 <instance part="R2" gate="G$1" x="86.36" y="45.72"/>
-<instance part="R3" gate="G$1" x="73.66" y="50.8" rot="R90"/>
+<instance part="R3" gate="G$1" x="73.66" y="68.58" rot="R270"/>
 <instance part="JP1" gate="G$1" x="25.4" y="63.5"/>
 <instance part="JP2" gate="G$1" x="109.22" y="58.42" rot="MR0"/>
-<instance part="GND1" gate="1" x="73.66" y="35.56"/>
+<instance part="SUPPLY1" gate="G$1" x="73.66" y="78.74"/>
 </instances>
 <busses>
@@
 <pinref part="R3" gate="G$1" pin="2"/>
 <wire x1="73.66" y1="60.96" x2="81.28" y2="60.96" width="0.1524" layer="91"/>
-<wire x1="73.66" y1="60.96" x2="73.66" y2="55.88" width="0.1524" layer="91"/>
+<wire x1="73.66" y1="60.96" x2="73.66" y2="63.5" width="0.1524" layer="91"/>
 <junction x="73.66" y="60.96"/>
 </segment>
@@
 </segment>
 </net>
-<net name="GND" class="0">
-<segment>
-<pinref part="R3" gate="G$1" pin="1"/>
-<pinref part="GND1" gate="1" pin="GND"/>
-<wire x1="73.66" y1="45.72" x2="73.66" y2="38.1" width="0.1524" layer="91"/>
-</segment>
-</net>
 <net name="N$6" class="0">
 <segment>
@@
 </segment>
 </net>
+<net name="+5V/2" class="0">
+<segment>
+<pinref part="SUPPLY1" gate="G$1" pin="+5V/2"/>
+<pinref part="R3" gate="G$1" pin="1"/>
+<wire x1="73.66" y1="73.66" x2="73.66" y2="76.2" width="0.1524" layer="91"/>
+</segment>
+</net>
