File: OP amp module/Absolute value circuit.sch (EAGLE design)
At the start: 9 parts, among them IC1 LM358N

Commit message: abs val circuit
Connections:
- net GND renamed +5V/2
Changed lines of the file:
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@@
 <part name="JP1" library="SparkFun" deviceset="M01" device="PTH"/>
 <part name="JP2" library="SparkFun" deviceset="M01" device="PTH"/>
-<part name="GND1" library="SparkFun" deviceset="GND" device=""/>
+<part name="SUPPLY1" library="supply2" deviceset="+5V/2" device=""/>
 </parts>
 <sheets>
@@
 <instance part="JP1" gate="G$1" x="25.4" y="63.5"/>
 <instance part="JP2" gate="G$1" x="109.22" y="58.42" rot="MR0"/>
-<instance part="GND1" gate="1" x="73.66" y="35.56"/>
+<instance part="SUPPLY1" gate="G$1" x="81.28" y="35.56"/>
 </instances>
 <busses>
@@
 </segment>
 </net>
-<net name="GND" class="0">
-<segment>
-<pinref part="R3" gate="G$1" pin="1"/>
-<pinref part="GND1" gate="1" pin="GND"/>
-<wire x1="73.66" y1="45.72" x2="73.66" y2="38.1" width="0.1524" layer="91"/>
-</segment>
-</net>
 <net name="N$6" class="0">
 <segment>
@@
 </segment>
 </net>
+<net name="+5V/2" class="0">
+<segment>
+<pinref part="R3" gate="G$1" pin="1"/>
+<wire x1="73.66" y1="45.72" x2="73.66" y2="30.48" width="0.1524" layer="91"/>
+<pinref part="SUPPLY1" gate="G$1" pin="+5V/2"/>
+<wire x1="73.66" y1="30.48" x2="81.28" y2="30.48" width="0.1524" layer="91"/>
+<wire x1="81.28" y1="30.48" x2="81.28" y2="33.02" width="0.1524" layer="91"/>
+</segment>
+</net>
