File: IOBoard/IOBoard.brd (EAGLE design)
At the start: 100 x 80 mm, 11 parts, among them K1 S202SE1, K2 S202SE1

Commit message: io board
Parts:
- added LED1: (no value), adafruit:LED3MM
- added R1, R3: 4k7, My Library:1/6W-RES
- D1: value 1N4004 -> 1N4148; device diode:DO41-10 -> My Library:DO34-5
- moved X1 5.68 mm to (45.7, 49.5)
Connections:
- new net GND: OK1.3
- new net N$1: LED1.K, OK1.1
- new net N$2: R1.2, X1.1
- new net N$3: D1.A, OK1.2, X1.2
- new net N$4: D1.C, LED1.A, R1.1
- new net N$5: OK1.4, R3.1
- new net VCC: R3.2
Changed lines of the file:
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@@
 <?xml version="1.0" encoding="utf-8"?>
 <!DOCTYPE eagle SYSTEM "eagle.dtd">
-<eagle version="6.5.0">
+<eagle version="6.2">
 <drawing>
 <settings>
@@
 <layer number="48" name="Document" color="7" fill="1" visible="yes" active="yes"/>
 <layer number="49" name="Reference" color="7" fill="1" visible="yes" active="yes"/>
+<layer number="50" name="dxf" color="7" fill="1" visible="no" active="yes"/>
 <layer number="51" name="tDocu" color="7" fill="1" visible="yes" active="yes"/>
 <layer number="52" name="bDocu" color="7" fill="1" visible="yes" active="yes"/>
+<layer number="53" name="tGND_GNDA" color="7" fill="9" visible="no" active="no"/>
+<layer number="54" name="bGND_GNDA" color="1" fill="9" visible="no" active="no"/>
+<layer number="56" name="wert" color="7" fill="1" visible="no" active="yes"/>
 <layer number="91" name="Nets" color="2" fill="1" visible="no" active="no"/>
 <layer number="92" name="Busses" color="1" fill="1" visible="no" active="no"/>
@@
 <layer number="97" name="Info" color="7" fill="1" visible="no" active="no"/>
 <layer number="98" name="Guide" color="6" fill="1" visible="no" active="no"/>
+<layer number="100" name="Muster" color="7" fill="1" visible="no" active="no"/>
+<layer number="101" name="Patch_Top" color="12" fill="4" visible="no" active="yes"/>
+<layer number="102" name="Vscore" color="7" fill="1" visible="no" active="yes"/>
+<layer number="103" name="tMap" color="7" fill="1" visible="no" active="yes"/>
+<layer number="104" name="Name" color="16" fill="1" visible="no" active="yes"/>
+<layer number="105" name="tPlate" color="7" fill="1" visible="no" active="yes"/>
+<layer number="106" name="bPlate" color="7" fill="1" visible="no" active="yes"/>
+<layer number="107" name="Crop" color="7" fill="1" visible="no" active="yes"/>
+<layer number="108" name="fp8" color="7" fill="1" visible="no" active="yes"/>
+<layer number="109" name="fp9" color="7" fill="1" visible="no" active="yes"/>
+<layer number="110" name="fp0" color="7" fill="1" visible="no" active="yes"/>
+<layer number="116" name="Patch_BOT" color="9" fill="4" visible="no" active="yes"/>
+<layer number="121" name="_tsilk" color="7" fill="1" visible="no" active="yes"/>
+<layer number="122" name="_bsilk" color="7" fill="1" visible="no" active="yes"/>
+<layer number="123" name="tTestmark" color="7" fill="1" visible="no" active="yes"/>
+<layer number="124" name="bTestmark" color="7" fill="1" visible="no" active="yes"/>
+<layer number="125" name="_tNames" color="7" fill="1" visible="no" active="yes"/>
+<layer number="131" name="tAdjust" color="7" fill="1" visible="no" active="yes"/>
+<layer number="132" name="bAdjust" color="7" fill="1" visible="no" active="yes"/>
+<layer number="144" name="Drill_legend" color="7" fill="1" visible="no" active="yes"/>
+<layer number="151" name="HeatSink" color="7" fill="1" visible="no" active="yes"/>
+<layer number="199" name="Contour" color="7" fill="1" visible="yes" active="yes"/>
+<layer number="200" name="200bmp" color="1" fill="10" visible="no" active="yes"/>
+<layer number="201" name="201bmp" color="2" fill="10" visible="no" active="yes"/>
+<layer number="202" name="202bmp" color="3" fill="10" visible="no" active="yes"/>
+<layer number="203" name="203bmp" color="4" fill="10" visible="no" active="yes"/>
+<layer number="204" name="204bmp" color="5" fill="10" visible="no" active="yes"/>
+<layer number="205" name="205bmp" color="6" fill="10" visible="no" active="yes"/>
+<layer number="206" name="206bmp" color="7" fill="10" visible="no" active="yes"/>
+<layer number="207" name="207bmp" color="8" fill="10" visible="no" active="yes"/>
+<layer number="208" name="208bmp" color="9" fill="10" visible="no" active="yes"/>
+<layer number="209" name="209bmp" color="7" fill="1" visible="no" active="yes"/>
+<layer number="210" name="210bmp" color="7" fill="1" visible="no" active="yes"/>
+<layer number="211" name="211bmp" color="7" fill="1" visible="no" active="yes"/>
+<layer number="212" name="212bmp" color="7" fill="1" visible="no" active="yes"/>
+<layer number="213" name="213bmp" color="7" fill="1" visible="no" active="yes"/>
+<layer number="214" name="214bmp" color="7" fill="1" visible="no" active="yes"/>
+<layer number="215" name="215bmp" color="7" fill="1" visible="no" active="yes"/>
+<layer number="216" name="216bmp" color="7" fill="1" visible="no" active="yes"/>
+<layer number="217" name="217bmp" color="18" fill="1" visible="no" active="no"/>
+<layer number="218" name="218bmp" color="19" fill="1" visible="no" active="no"/>
+<layer number="219" name="219bmp" color="20" fill="1" visible="no" active="no"/>
+<layer number="220" name="220bmp" color="21" fill="1" visible="no" active="no"/>
+<layer number="221" name="221bmp" color="22" fill="1" visible="no" active="no"/>
+<layer number="222" name="222bmp" color="23" fill="1" visible="no" active="no"/>
+<layer number="223" name="223bmp" color="24" fill="1" visible="no" active="no"/>
+<layer number="224" name="224bmp" color="25" fill="1" visible="no" active="no"/>
+<layer number="250" name="Descript" color="3" fill="1" visible="no" active="no"/>
+<layer number="251" name="SMDround" color="12" fill="11" visible="no" active="no"/>
+<layer number="254" name="cooling" color="7" fill="1" visible="no" active="yes"/>
 </layers>
 <board>
@@
 </class>
 </classes>
-<designrules name="default">
+<designrules>
 <description language="de">&lt;b&gt;EAGLE Design Rules&lt;/b&gt;
 &lt;p&gt;
@@
 <attribute name="OC_FARNELL" value="unknown" x="63.5" y="6.35" size="1.778" layer="27" display="off"/>
 </element>
-<element name="X1" library="con-wago-500" package="W237-6" value="" x="50.8" y="46.99">
-<attribute name="OC_NEWARK" value="unknown" x="78.74" y="10.16" size="1.778" layer="27" display="off"/>
-<attribute name="MPN" value="" x="78.74" y="10.16" size="1.778" layer="27" display="off"/>
-<attribute name="MF" value="" x="78.74" y="10.16" size="1.778" layer="27" display="off"/>
-<attribute name="OC_FARNELL" value="unknown" x="78.74" y="10.16" size="1.778" layer="27" display="off"/>
-</element>
-<element name="D1" library="diode" package="DO41-10" value="1N4004" x="77.47" y="50.8"/>
+<element name="X1" library="con-wago-500" package="W237-6" value="" x="45.72" y="49.53">
+<attribute name="OC_NEWARK" value="unknown" x="73.66" y="12.7" size="1.778" layer="27" display="off"/>
+<attribute name="MPN" value="" x="73.66" y="12.7" size="1.778" layer="27" display="off"/>
+<attribute name="MF" value="" x="73.66" y="12.7" size="1.778" layer="27" display="off"/>
+<attribute name="OC_FARNELL" value="unknown" x="73.66" y="12.7" size="1.778" layer="27" display="off"/>
+</element>
+<element name="D1" library="My Library" package="DO34-5" value="1N4148" x="77.47" y="50.8"/>
 <element name="D2" library="diode" package="DO41-10" value="1N4004" x="77.47" y="43.18"/>
 <element name="D3" library="diode" package="DO41-10" value="1N4004" x="76.2" y="35.56"/>
@@
 <element name="D4" library="diode" package="DO41-10" value="1N4004" x="6.35" y="-3.81"/>
 <element name="D5" library="diode" package="DO41-10" value="1N4004" x="6.35" y="-11.43"/>
+<element name="LED1" library="adafruit" package="LED3MM" value="" x="3.81" y="-24.13"/>
+<element name="R1" library="My Library" package="1/6W-RES" value="4k7" x="3.81" y="-29.21"/>
+<element name="R3" library="My Library" package="1/6W-RES" value="4k7" x="3.81" y="-36.83"/>
 </elements>
 <signals>
+<signal name="N$1">
+<contactref element="OK1" pad="1"/>
+<contactref element="LED1" pad="K"/>
+<wire x1="5.08" y1="-24.13" x2="27.94" y2="25.4" width="0" layer="19" extent="1-1"/>
+</signal>
+<signal name="N$2">
+<contactref element="R1" pad="2"/>
+<contactref element="X1" pad="1"/>
+<wire x1="6.31" y1="-29.21" x2="33.22" y2="48.26" width="0" layer="19" extent="1-1"/>
+</signal>
+<signal name="N$3">
+<contactref element="OK1" pad="2"/>
+<contactref element="X1" pad="2"/>
+<contactref element="D1" pad="A"/>
+<wire x1="38.22" y1="48.26" x2="80.01" y2="50.8" width="0" layer="19" extent="1-1"/>
+<wire x1="30.48" y1="25.4" x2="38.22" y2="48.26" width="0" layer="19" extent="1-1"/>
+</signal>
+<signal name="N$4">
+<contactref element="LED1" pad="A"/>
+<contactref element="R1" pad="1"/>
+<contactref element="D1" pad="C"/>
+<wire x1="2.54" y1="-24.13" x2="74.93" y2="50.8" width="0" layer="19" extent="1-1"/>
+<wire x1="1.31" y1="-29.21" x2="2.54" y2="-24.13" width="0" layer="19" extent="1-1"/>
+</signal>
+<signal name="GND">
+<contactref element="OK1" pad="3"/>
+</signal>
+<signal name="N$5">
+<contactref element="OK1" pad="4"/>
+<contactref element="R3" pad="1"/>
+<wire x1="1.31" y1="-36.83" x2="27.94" y2="33.02" width="0" layer="19" extent="1-1"/>
+</signal>
+<signal name="VCC">
+<contactref element="R3" pad="2"/>
+</signal>
 </signals>
 </board>
