File: IOBoard/IOBoard.sch (EAGLE design)
At the start: 11 parts, among them K1 S202SE1, K2 S202SE1

Commit message: io board
Parts:
- added LED1: (no value), adafruit:LED3MM
- added R1, R3: 4k7, My Library:RESISTORPTH-1/6W
- D1: value 1N4004 -> 1N4148; device diode:1N4004 -> My Library:1N4148
Connections:
- new net GND: OK1.EMIT
- new net N$1: LED1.C, OK1.A
- new net N$2: R1.2, X1-1.KL
- new net N$3: D1.A, OK1.C, X1-2.KL
- new net N$4: D1.C, LED1.A, R1.1
- new net N$5: OK1.COL, R3.1
- new net VCC: R3.2
Other:
- moved on the sheet: D2, X1-1, X1-2, X1-3, X1-4, X1-5, X1-6
