File: Quaranta/Arduino-R3-Board.brd (EAGLE design)
At the start: 100 x 80 mm, 7 parts, among them IC1 ATMEGA644A, U1 ARDUINOR3-BPLACE

Commit message: Quaranta
Parts:
- moved C3 32.7 mm to (71.1, 47.0), turned to 90 degrees
- moved C2 31.9 mm to (71.1, 41.9), turned to 270 degrees
- moved Q1 31.9 mm to (76.2, 44.5), turned to 270 degrees
- moved IC1 1.27 mm to (58.4, 44.5), turned to 180 degrees
Routing:
- net N$4: track 0.00 -> 36.3 mm
- net N$5: track 0.00 -> 32.9 mm
- net N$13: track 0.00 -> 11.5 mm
- net N$14: track 0.00 -> 9.44 mm
